File: modules/audio-codec/audio-codec.kicad_sch (KiCad schematic)
At the start: 24 parts, among them U1 TLV320AIC3110IRHBR, U2 ADP5301ACBZ-1-R7

Commit message: Updating all modules
Other:
- moved on the sheet: C2, C3, L1, R2, R3, U2
