File: modules/audio-jack/audio-jack.kicad_sch (KiCad schematic)
At the start: 6 parts, among them J1 SJ-43514-SMT-TR

Commit message: Updating all modules
Other:
- moved on the sheet: J1, JP1, JP2, JP3, JP4, M1
