File: modules/audio-jack/audio-jack.kicad_sch (KiCad schematic)
At the start: 6 parts, among them J1 SJ-43514-SMT-TR

Commit message: Updating all schematics
Other:
- note added: "${project_name} ${project_version} ${project_creator} License: ${project_license} Year: ${project_year}"
- note added: "......"
- note added: "......."
- note added: "1"
- note added: "3D top side"
- note added: "CoverPage"
- note added: "Index"
- note added: "Page"
- company: (none) -> ${project_creator}
- title: (none) -> ${project_name}
- moved on the sheet: J1, JP1, JP2, JP3, JP4, M1
