File: modules/bluetooth/bluetooth.kicad_sch (KiCad schematic)
At the start: 2 parts, among them U1 Microchip_BM83

Commit message: Updating all schematics
Other:
- note added: "${project_name} ${project_version} ${project_creator} License: ${project_license} Year: ${project_year}"
- note added: "......"
- note added: "......."
- note added: "1"
- note added: "3D top side"
- note added: "CoverPage"
- note added: "Index"
- note added: "Page"
- company: (none) -> ${project_creator}
- title: (none) -> ${project_name}
- moved on the sheet: M1, U1
