File: modules/high-efficiency_dc-dc_converter/high-efficiency_dc-dc_converter.kicad_sch (KiCad schematic)
At the start: 13 parts, among them U1 ISl91127IR

Commit message: Updating all schematics
Parts:
- added C6, C7: 10n, Capacitor_SMD:C_0603_1608Metric, symbol Device:C_Small
- added C8: 100n, Capacitor_SMD:C_0603_1608Metric, symbol Device:C_Small
- added C9: 2.2uF, Capacitor_SMD:C_0603_1608Metric, symbol Device:C_Small
- added R3: R0, Resistor_SMD:R_0603_1608Metric, symbol Device:R_Small
- added U2: RFM95W-868S2, RF_Module:HOPERF_RFM9XW_SMD, symbol RF_Module:RFM95W-868S2
Connections:
- net GND: now also C6.2, C7.2, C8.2, C9.2, U2.1 (GND), U2.10 (GND), U2.8 (GND)
- new net: C6.1, R3.1
- new net: R3.2, U2.9 (ANT)
- new net +3.3V: C7.1, C8.1, C9.1, U2.13 (3.3V)
Other:
- note added: "${project_name} ${project_version} ${project_creator} License: ${project_license} Year: ${project_year}"
- note added: "......"
- note added: "......."
- note added: "1"
- note added: "3D top side"
- note added: "CoverPage"
- note added: "Index"
- note added: "Page"
- company: (none) -> ${project_creator}
- title: High-Efficiency DC:DC Converter Module -> ${project_name}
- moved on the sheet: C1, C2, C3, C4, C5, JP1, L1, M1, R1, R2, R4, R5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

Commit message: Updating schematics
Parts:
- removed C6, C7: 10n, Capacitor_SMD:C_0603_1608Metric, symbol Device:C_Small
- removed C8: 100n, Capacitor_SMD:C_0603_1608Metric, symbol Device:C_Small
- removed C9: 2.2uF, Capacitor_SMD:C_0603_1608Metric, symbol Device:C_Small
- removed R3: R0, Resistor_SMD:R_0603_1608Metric, symbol Device:R_Small
- removed U2: RFM95W-868S2, RF_Module:HOPERF_RFM9XW_SMD, symbol RF_Module:RFM95W-868S2
Other:
- moved on the sheet: C1, C2, C3, C4, C5, JP1, L1, M1, R1, R2, R4, R5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
