File: modules/input-power-selector/input-power-selector.kicad_sch (KiCad schematic)
At the start: 37 parts, among them Q1 SI4909DY-T1-GE3, Q2 SI4909DY-T1-GE3, Q3 SI4909DY-T1-GE3, Q4 IPF067N20NM6ATMA1, Q7 BC847, U1 LTC4417IGN, U2 SQJQ141EL-T1_GE3

Commit message: Updating all schematics
Other:
- note added: "${project_name} ${project_version} ${project_creator} License: ${project_license} Year: ${project_year}"
- note added: "......"
- note added: "......."
- note added: "1"
- note added: "3D top side"
- note added: "CoverPage"
- note added: "Index"
- note added: "Page"
- company: (none) -> ${project_creator}
- title: (none) -> ${project_name}
- moved on the sheet: M2
Changed lines of the file:
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@@
 	(generator_version "9.0")
 	(paper "A4")
+	(title_block
+		(title "${project_name}")
+		(date "2025-11-10")
+		(rev "${project_version}")
+		(company "${project_creator}")
+		(comment 1 "${project_license}")
+	)
+	(rectangle
+		(start 226.568 12.7)
+		(end 282.448 48.26)
+		(stroke
+			(width 0)
+			(type default)
+		)
+		(fill
+			(type color)
+			(color 0 255 0 0.1)
+		)
+	)
+	(rectangle
+		(start -282.829 196.977)
+		(end -223.901 242.697)
+		(stroke
+			(width 0)
+			(type default)
+		)
+		(fill
+			(type color)
+			(color 0 255 0 0.1)
+		)
+	)
+	(rectangle
+		(start 13.462 13.462)
+		(end 82.169 28.956)
+		(stroke
+			(width 0)
+			(type solid)
+		)
+		(fill
+			(type color)
+			(color 58 146 255 1)
+		)
+	)
 	(text "For the resistor laddars on the input power sources to\nthe source selector, we need to get V_UV and V_OV = 1V\nat the respective ends of the acceptable voltage range.\n\nIf we aim for 5V -- 28V being acceptable, then we can\nuse 246K, 51K and 11K, from VIN to GND respectively."
 		(exclude_from_sim no)
@@
 		)
 	)
+	(text "3D top side"
+		(exclude_from_sim no)
+		(at -254.127 201.803 0)
+		(effects
+			(font
+				(size 3.81 3.81)
+				(thickness 0.762)
+				(bold yes)
+			)
+		)
+	)
 	(text "Filter on VOUT pin to protect against\nnegative transients if output side is shorted."
 		(exclude_from_sim no)
@@
 		)
 	)
+	(text "......"
+		(exclude_from_sim no)
+		(at 235.966 23.876 0)
+		(effects
+			(font
+				(size 3.81 3.81)
+				(thickness 0.762)
+				(bold yes)
+			)
+		)
+	)
+	(text "1"
+		(exclude_from_sim no)
+		(at 270.256 30.734 0)
+		(effects
+			(font
+				(size 3.81 3.81)
+			)
+			(href "#1")
+		)
+	)
+	(text "CoverPage"
+		(exclude_from_sim no)
+		(at 243.84 30.48 0)
+		(effects
+			(font
+				(size 3.81 3.81)
+			)
+			(href "#1")
+		)
+	)
+	(text "......"
+		(exclude_from_sim no)
+		(at 235.966 41.91 0)
+		(effects
+			(font
+				(size 3.81 3.81)
+				(thickness 0.762)
+				(bold yes)
+			)
+		)
+	)
 	(text "Reverse polarity protection (to 100V)\nfor Dirty DC / external solar panel."
 		(exclude_from_sim no)
-		(at 211.328 124.968 0)
+		(at 211.836 126.492 0)
 		(effects
 			(font
@@
 		)
 	)
+	(text "${project_name} ${project_version}\n${project_creator}\nLicense: ${project_license}\nYear: ${project_year}"
+		(exclude_from_sim no)
+		(at 15.24 15.24 0)
+		(effects
+			(font
+				(size 2.032 2.032)
+			)
+			(justify left top)
+		)
+	)
+	(text "Page"
+		(exclude_from_sim no)
+		(at 235.966 18.034 0)
+		(effects
+			(font
+				(size 3.81 3.81)
+				(thickness 0.762)
+				(bold yes)
+			)
+		)
+	)
+	(text "......."
+		(exclude_from_sim no)
+		(at 271.272 41.91 0)
+		(effects
+			(font
+				(size 3.81 3.81)
+				(thickness 0.762)
+				(bold yes)
+			)
+		)
+	)
+	(text "         Index"
+		(exclude_from_sim no)
+		(at 257.81 18.034 0)
+		(effects
+			(font
+				(size 3.81 3.81)
+				(thickness 0.762)
+				(bold yes)
+			)
+		)
+	)
+	(text "......."
+		(exclude_from_sim no)
+		(at 270.51 23.876 0)
+		(effects
+			(font
+				(size 3.81 3.81)
+				(thickness 0.762)
+				(bold yes)
+			)
+		)
+	)
 	(text "Over-voltage protection bypass"
 		(exclude_from_sim no)
@@
 	)
 	(no_connect
-		(at 238.76 40.64)
+		(at 217.17 54.61)
 	)
 	(wire
@@
 	(wire
 		(pts
-			(xy 252.73 99.06) (xy 254 99.06)
+			(xy 231.14 113.03) (xy 232.41 113.03)
 		)
 		(stroke
@@
 	(wire
 		(pts
-			(xy 236.22 99.06) (xy 238.76 99.06)
+			(xy 214.63 113.03) (xy 217.17 113.03)
 		)
 		(stroke
@@
 	(global_label "DIRTY_DC_+"
 		(shape input)
-		(at 252.73 50.8 0)
+		(at 231.14 64.77 0)
 		(fields_autoplaced yes)
 		(effects
@@
 		)
 		(property "Intersheetrefs" "${INTERSHEET_REFS}"
-			(at 266.9638 50.8 0)
+			(at 245.3738 64.77 0)
 			(effects
 				(font
@@
 	(global_label "ENABLE"
 		(shape input)
-		(at 238.76 93.98 180)
+		(at 217.17 107.95 180)
 		(fields_autoplaced yes)
 		(effects
@@
 		)
 		(property "Intersheetrefs" "${INTERSHEET_REFS}"
-			(at 228.7596 93.98 0)
+			(at 207.1696 107.95 0)
 			(effects
 				(font
@@
 	(global_label "{slash}VALID1"
 		(shape output)
-		(at 238.76 88.9 180)
+		(at 217.17 102.87 180)
 		(fields_autoplaced yes)
 		(effects
@@
 		)
 		(property "Intersheetrefs" "${INTERSHEET_REFS}"
-			(at 228.1547 88.9 0)
+			(at 206.5647 102.87 0)
 			(effects
 				(font
@@
 	(global_label "USB-C_POWER_IN"
 		(shape input)
-		(at 238.76 60.96 180)
+		(at 217.17 74.93 180)
 		(fields_autoplaced yes)
 		(effects
@@
 		)
 		(property "Intersheetrefs" "${INTERSHEET_REFS}"
-			(at 218.781 60.96 0)
+			(at 197.191 74.93 0)
 			(effects
 				(font
@@
 	(global_label "{slash}SHUTDOWN"
 		(shape input)
-		(at 238.76 91.44 180)
+		(at 217.17 105.41 180)
 		(fields_autoplaced yes)
 		(effects
@@
 		)
 		(property "Intersheetrefs" "${INTERSHEET_REFS}"
-			(at 224.2238 91.44 0)
+			(at 202.6338 105.41 0)
 			(effects
 				(font
@@
 	(global_label "VOUT"
 		(shape output)
-		(at 238.76 50.8 180)
+		(at 217.17 64.77 180)
 		(fields_autoplaced yes)
 		(effects
@@
 		)
 		(property "Intersheetrefs" "${INTERSHEET_REFS}"
-			(at 231.0576 50.8 0)
+			(at 209.4676 64.77 0)
 			(effects
 				(font
@@
 	(global_label "VOUT"
 		(shape output)
-		(at 252.73 40.64 0)
+		(at 231.14 54.61 0)
 		(fields_autoplaced yes)
 		(effects
@@
 		)
 		(property "Intersheetrefs" "${INTERSHEET_REFS}"
-			(at 260.4324 40.64 0)
+			(at 238.8424 54.61 0)
 			(effects
 				(font
@@
 	(global_label "{slash}VALID3"
 		(shape output)
-		(at 238.76 83.82 180)
+		(at 217.17 97.79 180)
 		(fields_autoplaced yes)
 		(effects
@@
 		)
 		(property "Intersheetrefs" "${INTERSHEET_REFS}"
-			(at 228.1547 83.82 0)
+			(at 206.5647 97.79 0)
 			(effects
 				(font
@@
 	(global_label "{slash}VALID2"
 		(shape output)
-		(at 238.76 86.36 180)
+		(at 217.17 100.33 180)
 		(fields_autoplaced yes)
 		(effects
@@
 		)
 		(property "Intersheetrefs" "${INTERSHEET_REFS}"
-			(at 228.1547 86.36 0)
+			(at 206.5647 100.33 0)
 			(effects
 				(font
@@
 	(global_label "DIRTY_DC_-"
 		(shape input)
-		(at 252.73 53.34 0)
+		(at 231.14 67.31 0)
 		(fields_autoplaced yes)
 		(effects
@@
 		)
 		(property "Intersheetrefs" "${INTERSHEET_REFS}"
-			(at 266.9638 53.34 0)
+			(at 245.3738 67.31 0)
 			(effects
 				(font
@@
 	(global_label "INTERNAL_SOLAR_IN"
 		(shape input)
-		(at 238.76 71.12 180)
+		(at 217.17 85.09 180)
 		(fields_autoplaced yes)
 		(effects
@@
 		)
 		(property "Intersheetrefs" "${INTERSHEET_REFS}"
-			(at 217.2085 71.12 0)
+			(at 195.6185 85.09 0)
 			(effects
 				(font
@@
 	(symbol
 		(lib_id "power:GND")
-		(at 254 99.06 0)
+		(at 232.41 113.03 0)
 		(unit 1)
 		(exclude_from_sim no)
@@
 		(fields_autoplaced yes)
 		(property "Reference" "#PWR20"
-			(at 254 105.41 0)
+			(at 232.41 119.38 0)
 			(effects
 				(font
@@
 		)
 		(property "Value" "GND"
-			(at 254 104.14 0)
+			(at 232.41 118.11 0)
 			(effects
 				(font
@@
 		)
 		(property "Footprint" ""
-			(at 254 99.06 0)
+			(at 232.41 113.03 0)
 			(effects
 				(font
@@
 		)
 		(property "Datasheet" ""
-			(at 254 99.06 0)
+			(at 232.41 113.03 0)
 			(effects
 				(font
@@
 		)
 		(property "Description" "Power symbol creates a global label with name \"GND\" , ground"
-			(at 254 99.06 0)
+			(at 232.41 113.03 0)
 			(effects
 				(font
@@
 	(symbol
 		(lib_id "power:GND")
-		(at 236.22 99.06 0)
+		(at 214.63 113.03 0)
 		(unit 1)
 		(exclude_from_sim no)
@@
 		(fields_autoplaced yes)
 		(property "Reference" "#PWR19"
-			(at 236.22 105.41 0)
+			(at 214.63 119.38 0)
 			(effects
 				(font
@@
 		)
 		(property "Value" "GND"
-			(at 236.22 104.14 0)
+			(at 214.63 118.11 0)
 			(effects
 				(font
@@
 		)
 		(property "Footprint" ""
-			(at 236.22 99.06 0)
+			(at 214.63 113.03 0)
 			(effects
 				(font
@@
 		)
 		(property "Datasheet" ""
-			(at 236.22 99.06 0)
+			(at 214.63 113.03 0)
 			(effects
 				(font
@@
 		)
 		(property "Description" "Power symbol creates a global label with name \"GND\" , ground"
-			(at 236.22 99.06 0)
+			(at 214.63 113.03 0)
 			(effects
 				(font
@@
 	(symbol
 		(lib_id "MegaCastle:MegaCastle2x24-Module-I42.0x56.2-M88887D8C0001")
-		(at 245.11 69.85 0)
+		(at 223.52 83.82 0)
 		(unit 1)
 		(exclude_from_sim no)
@@
 		(fields_autoplaced yes)
 		(property "Reference" "M2"
-			(at 245.745 35.56 0)
+			(at 224.155 49.53 0)
 			(effects
 				(font
@@
 		)
 		(property "Value" "~"
-			(at 245.745 36.83 0)
+			(at 224.155 50.8 0)
 			(effects
 				(font
@@
 		)
 		(property "Footprint" "MegaCastle:MegaCastle2x24-Module-I47.0x56.2-M88887D8C0001-SPAREPAD"
-			(at 245.11 106.68 0)
+			(at 223.52 120.65 0)
 			(effects
 				(font
@@
 		)
 		(property "Datasheet" ""
-			(at 245.11 64.77 0)
+			(at 223.52 78.74 0)
 			(effects
 				(font
@@
 		)
 		(property "Description" "Generated using footprint-gen .. 42 55 14 M88887D8C0001"
-			(at 245.11 69.85 0)
+			(at 223.52 83.82 0)
 			(effects
 				(font
