File: modules/solar-and-dc-connectors/solar-and-dc-connectors.kicad_sch (KiCad schematic)
At the start: 3 parts, among them J1 S2B-PH-K-SLFSN, J2 54-00127

Commit message: Updating all schematics
Other:
- note added: "${project_name} ${project_version} ${project_creator} License: ${project_license} Year: ${project_year}"
- note added: "......"
- note added: "......."
- note added: "1"
- note added: "3D top side"
- note added: "CoverPage"
- note added: "Index"
- note added: "Page"
- company: (none) -> ${project_creator}
- title: (none) -> ${project_name}
- moved on the sheet: J1, J2, M1
