File: modules/te0725-carrier/te0725-carrier.kicad_sch (KiCad schematic)
At the start: 3 parts, among them J1 Conn_02x25_Odd_Even, J2 Conn_02x25_Odd_Even

Commit message: Updating all modules
Other:
- moved on the sheet: J1, J2, M1
