File: modules/usb-c-power-in/usb-c-power-in.kicad_sch (KiCad schematic)
At the start: 2 parts, among them J1 Conn_01x02

Commit message: Updating all schematics
Other:
- note added: "${project_name} ${project_version} ${project_creator} License: ${project_license} Year: ${project_year}"
- note added: "......"
- note added: "......."
- note added: "1"
- note added: "3D top side"
- note added: "CoverPage"
- note added: "Index"
- note added: "Page"
- company: (none) -> ${project_creator}
- title: (none) -> ${project_name}
- moved on the sheet: J1, M1
Changed lines of the file:
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@@
 	(generator_version "9.0")
 	(paper "A4")
+	(title_block
+		(title "${project_name}")
+		(date "2025-11-10")
+		(rev "${project_version}")
+		(company "${project_creator}")
+		(comment 1 "${project_license}")
+	)
+	(rectangle
+		(start 224.282 16.51)
+		(end 280.162 62.23)
+		(stroke
+			(width 0)
+			(type default)
+		)
+		(fill
+			(type color)
+			(color 0 255 0 0.1)
+		)
+	)
+	(rectangle
+		(start 14.224 150.114)
+		(end 73.152 195.834)
+		(stroke
+			(width 0)
+			(type default)
+		)
+		(fill
+			(type color)
+			(color 0 255 0 0.1)
+		)
+	)
+	(rectangle
+		(start 14.986 15.24)
+		(end 73.406 30.734)
+		(stroke
+			(width 0)
+			(type solid)
+		)
+		(fill
+			(type color)
+			(color 58 146 255 1)
+		)
+	)
+	(text "3D top side"
+		(exclude_from_sim no)
+		(at 42.926 154.94 0)
+		(effects
+			(font
+				(size 3.81 3.81)
+				(thickness 0.762)
+				(bold yes)
+			)
+		)
+	)
+	(text "......"
+		(exclude_from_sim no)
+		(at 233.68 27.686 0)
+		(effects
+			(font
+				(size 3.81 3.81)
+				(thickness 0.762)
+				(bold yes)
+			)
+		)
+	)
+	(text "1"
+		(exclude_from_sim no)
+		(at 267.97 34.544 0)
+		(effects
+			(font
+				(size 3.81 3.81)
+			)
+			(href "#1")
+		)
+	)
 	(text "These USB-C Power Delivery modules that are available on AliExpress, \nAmazon and lots of other places are pretty good, but more variable than\nthe share-price of snake oil.\n\nWATCH ESPECIALLY FOR POLARITY SWITCHING OF THE POWER OUTPUT PINS!\n\nYou shouldn't need to change anything on this schematic, as it really\nis just connecting the power and GND pins. To support other variants\nyou will instead need to go to the PCB layout, and select the footprint\nthere and then press E, and then select \"open in footprint editor\" to\nmunge it to suit your module."
 		(exclude_from_sim no)
-		(at 49.53 48.514 0)
+		(at 100.33 76.454 0)
 		(effects
 			(font
@@
 		)
 	)
+	(text "CoverPage"
+		(exclude_from_sim no)
+		(at 241.554 34.29 0)
+		(effects
+			(font
+				(size 3.81 3.81)
+			)
+			(href "#1")
+		)
+	)
+	(text "......"
+		(exclude_from_sim no)
+		(at 233.68 45.72 0)
+		(effects
+			(font
+				(size 3.81 3.81)
+				(thickness 0.762)
+				(bold yes)
+			)
+		)
+	)
+	(text "${project_name} ${project_version}\n${project_creator}\nLicense: ${project_license}\nYear: ${project_year}"
+		(exclude_from_sim no)
+		(at 16.764 17.018 0)
+		(effects
+			(font
+				(size 2.032 2.032)
+			)
+			(justify left top)
+		)
+	)
+	(text "Page"
+		(exclude_from_sim no)
+		(at 233.68 21.844 0)
+		(effects
+			(font
+				(size 3.81 3.81)
+				(thickness 0.762)
+				(bold yes)
+			)
+		)
+	)
+	(text "......."
+		(exclude_from_sim no)
+		(at 268.986 45.72 0)
+		(effects
+			(font
+				(size 3.81 3.81)
+				(thickness 0.762)
+				(bold yes)
+			)
+		)
+	)
+	(text "         Index"
+		(exclude_from_sim no)
+		(at 255.524 21.844 0)
+		(effects
+			(font
+				(size 3.81 3.81)
+				(thickness 0.762)
+				(bold yes)
+			)
+		)
+	)
+	(text "......."
+		(exclude_from_sim no)
+		(at 268.224 27.686 0)
+		(effects
+			(font
+				(size 3.81 3.81)
+				(thickness 0.762)
+				(bold yes)
+			)
+		)
+	)
 	(no_connect
-		(at 74.93 97.79)
+		(at 125.73 125.73)
 	)
 	(no_connect
-		(at 60.96 69.85)
+		(at 111.76 97.79)
 	)
 	(no_connect
-		(at 74.93 69.85)
+		(at 125.73 97.79)
 	)
 	(global_label "GND"
 		(shape input)
-		(at 60.96 100.33 180)
+		(at 111.76 128.27 180)
 		(fields_autoplaced yes)
 		(effects
@@
 		)
 		(property "Intersheetrefs" "${INTERSHEET_REFS}"
-			(at 54.1043 100.33 0)
+			(at 104.9043 128.27 0)
 			(effects
 				(font
@@
 	(global_label "+20V"
 		(shape input)
-		(at 101.6 66.04 180)
+		(at 152.4 93.98 180)
 		(fields_autoplaced yes)
 		(effects
@@
 		)
 		(property "Intersheetrefs" "${INTERSHEET_REFS}"
-			(at 93.5348 66.04 0)
+			(at 144.3348 93.98 0)
 			(effects
 				(font
@@
 	(global_label "GND"
 		(shape input)
-		(at 101.6 68.58 180)
+		(at 152.4 96.52 180)
 		(fields_autoplaced yes)
 		(effects
@@
 		)
 		(property "Intersheetrefs" "${INTERSHEET_REFS}"
-			(at 94.7443 68.58 0)
+			(at 145.5443 96.52 0)
 			(effects
 				(font
@@
 	(global_label "+20V"
 		(shape input)
-		(at 74.93 100.33 0)
+		(at 125.73 128.27 0)
 		(fields_autoplaced yes)
 		(effects
@@
 		)
 		(property "Intersheetrefs" "${INTERSHEET_REFS}"
-			(at 82.9952 100.33 0)
+			(at 133.7952 128.27 0)
 			(effects
 				(font
@@
 	(symbol
 		(lib_id "MegaCastle:MegaCastle2x13-Module-I14.0x28.2-M800C00C-NOCUTOUT-EDGE")
-		(at 67.31 85.09 0)
+		(at 118.11 113.03 0)
 		(unit 1)
 		(exclude_from_sim no)
@@
 		(fields_autoplaced yes)
 		(property "Reference" "M1"
-			(at 67.8138 60.96 0)
+			(at 118.6138 88.9 0)
 			(effects
 				(font
@@
 		)
 		(property "Value" "~"
-			(at 67.8138 63.5 0)
+			(at 118.6138 91.44 0)
 			(effects
 				(font
@@
 		)
 		(property "Footprint" "MegaCastle:MegaCastle2x13-Module-I20.0x28.2-M800C00C-SPAREPAD"
-			(at 67.31 107.95 0)
+			(at 118.11 135.89 0)
 			(effects
 				(font
@@
 		)
 		(property "Datasheet" ""
-			(at 67.31 80.01 0)
+			(at 118.11 107.95 0)
 			(effects
 				(font
@@
 		)
 		(property "Description" "Generated using footprint-gen .. 14 28 5 M800C00C"
-			(at 67.31 85.09 0)
+			(at 118.11 113.03 0)
 			(effects
 				(font
@@
 	(symbol
 		(lib_id "Connector_Generic:Conn_01x02")
-		(at 106.68 66.04 0)
+		(at 157.48 93.98 0)
 		(unit 1)
 		(exclude_from_sim no)
@@
 		(fields_autoplaced yes)
 		(property "Reference" "J1"
-			(at 109.22 66.0399 0)
+			(at 160.02 93.9799 0)
 			(effects
 				(font
@@
 		)
 		(property "Value" "Conn_01x02"
-			(at 109.22 68.5799 0)
+			(at 160.02 96.5199 0)
 			(effects
 				(font
@@
 		)
 		(property "Footprint" "Connector_PinHeader_2.54mm:PinHeader_1x02_P2.54mm_Vertical"
-			(at 106.68 66.04 0)
+			(at 157.48 93.98 0)
 			(effects
 				(font
@@
 		)
 		(property "Datasheet" "~"
-			(at 106.68 66.04 0)
+			(at 157.48 93.98 0)
 			(effects
 				(font
@@
 		)
 		(property "Description" "Generic connector, single row, 01x02, script generated (kicad-library-utils/schlib/autogen/connector/)"
-			(at 106.68 66.04 0)
-			(effects
-				(font
+			(at 157.48 93.98 0)
+			(effects
+				(font
