File: modules/lcd-panel/lcd-panel.kicad_sch (KiCad schematic)
At the start: 10 parts, among them J1 5051100692, J2 5051104091, U1 LP8556SQ-E09/NOPB

Commit message: Updating all schematics
Other:
- note added: "${project_name} ${project_version} ${project_creator} License: ${project_license} Year: ${project_year}"
- note added: "......"
- note added: "......."
- note added: "1"
- note added: "3D top side"
- note added: "CoverPage"
- note added: "Index"
- note added: "Page"
- company: (none) -> ${project_creator}
- title: (none) -> ${project_name}
- moved on the sheet: C1, C2, C3, D1, L1, M2, R1, U1
