File: modules/lcd-panel/lcd-panel.kicad_pcb (KiCad board)
At the start: 4 copper layers, 40 x 91.4 mm, 10 parts, among them J1 5051100692, J2 5051104091, U1 LP8556SQ-E09/NOPB

Commit message: All updates in v1.1
Parts:
- moved J1 1.50 mm to (176.1, 133.6)
Routing:
- net GND: track 29.4 -> 27.4 mm, vias 120 -> 126
- net CTP_INT: track 22.5 -> 24.0 mm
- net CTP_GND: track 24.4 -> 25.9 mm
- net CPT_WAKE: track 21.0 -> 22.4 mm
- net CPT_VDD: track 19.0 -> 20.4 mm
- net CPT_SDA: track 17.2 -> 18.4 mm
- net CPT_SCL: track 15.4 -> 16.5 mm
- net RESIST_YD: track 32.1 -> 32.9 mm
- net RESIST_XL: track 32.6 -> 33.4 mm
