File: modules/megaphone-low-current-dc-dc-converter/megaphone-low-current-dc-dc-converter.kicad_sch (KiCad schematic)
At the start: 9 parts, among them U1 TPS631000DRLR

Commit message: Updating all modules
Other:
- moved on the sheet: C0, C1, L1, M2, R1, R2, R3, R4, U1

Commit message: Updating all schematics
Other:
- note added: "${project_name} ${project_version} ${project_creator} License: ${project_license} Year: ${project_year}"
- note added: "......"
- note added: "......."
- note added: "1"
- note added: "3D top side"
- note added: "CoverPage"
- note added: "Index"
- note added: "Page"
- company: (none) -> ${project_creator}
- title: MEGAphone megaphone-low-current-dc-dc-converter -> ${project_name}
- moved on the sheet: C0, C1, L1, M2, R1, R2, R3, R4, U1
