File: modules/mppt-charge-controller/MPPT Charge Controller.kicad_sch (KiCad schematic)
At the start: 53 parts, among them Q1 SI7272DP, Q3 2N7002, U2 AP63203WU, U3 ACS712, U4 ACS712, U5 MCP4018

Commit message: Updating all modules
Other:
- moved on the sheet: C11, C12, C13, C14, L2, U2

Commit message: Updating all schematics
Other:
- note added: "${project_name} ${project_version} ${project_creator} License: ${project_license} Year: ${project_year}"
- company: (none) -> ${project_creator}
- title: MEGAphone MPPT Charge Controller -> ${project_name}
- moved on the sheet: A1, C1, C10, C11, C12, C13, C14, C15, C2, C3, C4, C5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
