File: modules/main-carrier/main-carrier.kicad_pcb (KiCad board)
At the start: 4 copper layers, 311.8 x 203.2 mm, 29 parts

Commit message: Adding icesugar module - placing Ice sugar on base board, remove FPGA as module, add FPGA directly
Parts:
- removed M2: ~, MegaCastle:MegaCastle2x52-I42.0x127.3-M1
- added J1: Conn_01x06_Pin, Connector_PinHeader_2.54mm:PinHeader_1x06_P2.54mm_Vertical, F.Cu at (160.6, 256.4)
- added J2: Conn_01x06_Pin, Connector_PinHeader_2.54mm:PinHeader_1x06_P2.54mm_Vertical, F.Cu at (145.3, 243.7)
- added J3: Conn_02x06_Odd_Even, Connector_PinHeader_2.54mm:PinHeader_2x06_P2.54mm_Vertical, F.Cu at (159.3, 262.2)
- added J4: Conn_02x25_Odd_Even, Connector_PinHeader_2.54mm:PinHeader_2x25_P2.54mm_Vertical, F.Cu at (136.5, 140.5)
- added J5: Conn_02x25_Odd_Even, Connector_PinHeader_2.54mm:PinHeader_2x25_P2.54mm_Vertical, F.Cu at (164.4, 148.1)
- moved M5 74.5 mm to (212.7, 273.4)
- moved M1 21.6 mm to (323.4, 158.9)
- moved M12 21.6 mm to (382.4, 222.5)
- moved M11 21.6 mm to (383.2, 153.9)
- moved M14 21.6 mm to (380.1, 278.5)
- moved M8 21.6 mm to (312.0, 223.8)
- moved M10 21.6 mm to (342.9, 277.2)
- moved M13 21.6 mm to (309.5, 262.0)
- moved M9 21.6 mm to (346.2, 222.5)
Connections:
- net 3.5MM_LEFT renamed /3.5MM_LEFT
- net 3.5MM_MIC renamed /3.5MM_MIC
- net 3.5MM_RIGHT renamed /3.5MM_RIGHT
- M1 pad 22: USIM_VDD -> /USIM_VDD
- M1 pad 23: unconnected-(M1-Pad23) -> /USIM_DATA
- M1 pad 24: USIM_CLK -> /USIM_CLK
- M1 pad 25: unconnected-(M1-Pad25) -> //USIM_RESET
- M1 pad 26: USIM_VPP -> /USIM_VPP
- M1 pad 35: PCM_DIN_3V3 -> J1_13
- M1 pad 42: PCM_CLK_3V3 -> J1_27
- M1 pad 43: PCM_SYNC_3V# -> J1_29
- M1 pad 44: PCM_CLK_DIR -> J1_31
- M10 pad 11: SD_DAT2 -> J2_10
- M10 pad 13: SIM_CLK -> /USIM_CLK
- M10 pad 14: SIM_DATA -> /USIM_DATA
- M10 pad 15: SD_CLK -> J2_8
- M10 pad 17: SD_GND -> GND
- M10 pad 18: SD_DAT0 -> J2_6
- M10 pad 19: SD_PRESENT -> J2_4
- M10 pad 20: SD_DAT1 -> J2_2
- M10 pad 3: SIM_VCC -> /USIM_VDD
- M10 pad 4: SIM_RESET -> //USIM_RESET
- M10 pad 5: SIM_VPP -> /USIM_VPP
- M10 pad 7: SIM_GND -> GND
- M10 pad 8: SD_CMD -> J2_12
- M10 pad 9: SD_CD -> J2_14
- M12 pad 15: SDA -> J1_14
- M12 pad 16: SCL -> J1_12
- M12 pad 19: PWM -> J2_34
- M14 pad 17: WCLK -> J1_20
- M14 pad 20: SDA -> J1_14
- M14 pad 21: SCL -> J1_12
- M14 pad 4: V1.8_MODE -> J1_26
- M15 pad 1: VBAT_+ -> VBAT_OUT
- M15 pad 5: VBAT_- -> GND
- M3 pad 1: VBAT_OUT -> unconnected-(M3-VCC-Pad1)
- M4 pad 10: SWDIO -> J2_42
- M4 pad 32: SCL -> unconnected-(M4-Pad32)
- M4 pad 33: SDA -> unconnected-(M4-Pad33)
- M4 pad 9: SWCLK -> J2_40
- M5 pad 15: MODE -> J1_8
- M5 pad 16: SEL1V8 -> J1_6
- M6 pad 20: VSYNC -> J2_39
- M6 pad 51: RED5 -> J2_32
- M6 pad 52: RED6 -> J2_30
- M6 pad 53: RED7 -> J2_28
- M7 pad 4: LR_SELECT -> J1_32
- M8 pad 26: +20V -> USB-C_POWER_IN
- M9 pad 24: INTERNAL_SOLAR_+ -> INTERNAL_SOLAR_IN
Routing:
- net J1_46: vias 0 -> 1
Other:
- board text added: "3.3V"
- board text added: "A1"
- board text added: "A1'"
- board text added: "A3"
- board text added: "B1"
- board text added: "B1'"
- board text added: "B3"
- board text added: "B4"
- board text added: "B5"
- board text added: "B6"
- board text added: "C2"
- board text added: "C5"
- board text added: "C6"
- board text added: "D1"
- board text added: "E1"
- board text added: "E2"
- board text added: "E3"
- board text added: "GND"
- board text added: "MEGAphone iCESugar Nano Carrier 20250806 REMOVE U6, bridge with diode to power from 3.3V If not, 3.3V is OUTPUT not INPUT!!!"

Commit message: Routing
Parts:
- removed LOGO1: Intergalaktik Logo, intergalaktik:intergalaktik
- removed LOGO2: Radiona Logo, radiona:radiona
- added D2: LED_Small, LED_SMD:LED_0603_1608Metric, F.Cu at (414.5, 133.1)
- added D3: LED_Small, LED_SMD:LED_0603_1608Metric, F.Cu at (414.4, 134.9)
- added H5: MH, MountingHole:MountingHole_3mm_Pad, F.Cu at (132.0, 107.6)
- added H6: MH, MountingHole:MountingHole_3mm_Pad, F.Cu at (262.0, 107.6)
- added H7: MH, MountingHole:MountingHole_3mm_Pad, F.Cu at (132.0, 182.6)
- added H8: MH, MountingHole:MountingHole_3mm_Pad, F.Cu at (262.0, 182.6)
- added IC1: PCA9535DW, PCA9535DW:SOIC127P1030X265-24N, F.Cu at (340.0, 174.2)
- added IC2: PCA9535DW, PCA9535DW:SOIC127P1030X265-24N, F.Cu at (278.5, 252.1)
- added IC3: PCA9535DW, PCA9535DW:SOIC127P1030X265-24N, F.Cu at (400.8, 164.1)
- added J10: CELULAR_3V3, Connector_PinSocket_2.54mm:PinSocket_1x02_P2.54mm_Vertical, F.Cu at (263.7, 118.4)
- added J11: LORA_3V3, Connector_PinSocket_2.54mm:PinSocket_1x02_P2.54mm_Vertical, F.Cu at (377.2, 114.9)
- added J12: AudioCDC_VCC, Connector_PinSocket_2.54mm:PinSocket_1x03_P2.54mm_Vertical, F.Cu at (271.4, 195.1)
- added J13: SD_VCC, Connector_PinSocket_2.54mm:PinSocket_1x03_P2.54mm_Vertical, F.Cu at (244.8, 194.6)
- added J14: SIM_VCC, Connector_PinSocket_2.54mm:PinSocket_1x03_P2.54mm_Vertical, F.Cu at (230.1, 194.9)
- added J15: LORA_BAT, Connector_PinSocket_2.54mm:PinSocket_1x02_P2.54mm_Vertical, F.Cu at (324.7, 114.1)
- added J16: I2C1_VCC, Connector_PinSocket_2.54mm:PinSocket_1x03_P2.54mm_Vertical, F.Cu at (266.2, 254.3)
- added J17: FPGA_VCCIO, Connector_PinSocket_2.54mm:PinSocket_1x03_P2.54mm_Vertical, F.Cu at (201.3, 250.4)
- added J18: I2C1_VCC, Connector_PinSocket_2.54mm:PinSocket_1x03_P2.54mm_Vertical, F.Cu at (411.8, 156.0)
- added J19: I2C1_VCC, Connector_PinSocket_2.54mm:PinSocket_1x03_P2.54mm_Vertical, F.Cu at (323.2, 171.9)
- added J21: UART_CELL, Connector_PinSocket_2.54mm:PinSocket_1x02_P2.54mm_Vertical, F.Cu at (263.4, 155.3)
- added J6: Mic_VCC, Connector_PinSocket_2.54mm:PinSocket_1x03_P2.54mm_Vertical, F.Cu at (195.9, 275.8)
- added J7: AudioCDC_VBAT, Connector_PinSocket_2.54mm:PinSocket_1x02_P2.54mm_Vertical, F.Cu at (262.2, 207.7)
- added J8: BT_3V3, Connector_PinSocket_2.54mm:PinSocket_1x02_P2.54mm_Vertical, F.Cu at (374.6, 119.1)
- added J9: LCD_3V3, Connector_PinSocket_2.54mm:PinSocket_1x02_P2.54mm_Vertical, F.Cu at (219.6, 195.7)
- added Q1: BSS138, Package_TO_SOT_SMD:SOT-23, F.Cu at (148.5, 280.5)
- added Q2: BSS138, Package_TO_SOT_SMD:SOT-23, F.Cu at (153.8, 280.5)
- added R2: 10K, Resistor_SMD:R_0603_1608Metric, F.Cu at (152.3, 278.0)
- added R3: 10K, Resistor_SMD:R_0603_1608Metric, F.Cu at (155.2, 278.0)
- added R4: 10K, Resistor_SMD:R_0603_1608Metric, F.Cu at (147.0, 277.9)
- added R5: 10K, Resistor_SMD:R_0603_1608Metric, F.Cu at (149.9, 278.0)
- added R6: 10K, Resistor_SMD:R_0603_1608Metric, F.Cu at (414.5, 131.3)
- added R7: 10K, Resistor_SMD:R_0603_1608Metric, F.Cu at (414.5, 136.5)
- moved R1 200.7 mm to (286.6, 247.4)
- moved M3 191.1 mm to (388.1, 208.9)
- moved M4 169.3 mm to (349.4, 134.9)
- moved D1 158.1 mm to (287.1, 245.2), turned to -90 degrees
- moved J4 148.0 mm to (128.9, 288.3), turned to 90 degrees
- moved M14 118.7 mm to (278.6, 216.8)
- moved M10 117.1 mm to (243.2, 215.8)
- moved J5 115.7 mm to (136.5, 260.4), turned to 90 degrees
- moved J2 108.1 mm to (246.9, 280.6), turned to 180 degrees
- moved M6 105.8 mm to (171.4, 224.8), turned to -90 degrees
- moved M8 101.7 mm to (402.9, 269.5), turned to 180 degrees
- moved M15 100.0 mm to (339.1, 288.3)
- moved M12 97.6 mm to (394.8, 125.7)
- moved M11 87.7 mm to (329.1, 222.9)
- moved M5 84.5 mm to (296.6, 283.5), turned to 180 degrees
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Connections:
- net B4 renamed B4_FPGA
- net B5 renamed B5_FPGA
- net BLUE0 renamed /BLUE0
- net BLUE1 renamed /BLUE1
- net BLUE2 renamed /BLUE2
- net BLUE3 renamed /BLUE3
- net C2 renamed C2_FPGA
- net C6 renamed C6_FPGA
- net CTP_GND renamed /CTP_GND
- net DECOUPLE5 renamed /DECOUPLE5
- net E1 renamed E1_FPGA
- net E3 renamed E3_FPGA
- net GREEN0 renamed /GREEN0
- net GREEN1 renamed /GREEN1
- net GREEN2 renamed /GREEN2
- net GREEN3 renamed /GREEN3
- net RED0 renamed /RED0
- net RED1 renamed /RED1
- net RED2 renamed /RED2
- net RED3 renamed /RED3
- net RESIST_XL renamed /RESIST_XL
- net RESIST_XR renamed /RESIST_XR
- net RESIST_YD renamed /RESIST_YD
- net RESIST_YU renamed /RESIST_YU
- net SPEAKER_L_M renamed /SPEAKER_L_M
- net SPEAKER_L_P renamed /SPEAKER_L_P
- net SPEAKER_R_M renamed /SPEAKER_R_M
- net SPEAKER_R_P renamed /SPEAKER_R_P
- J1 pad 1: B3 -> B3_FPGA
- J1 pad 2: A3 -> A3_FPGA
- J1 pad 3: B6 -> B6_FPGA
- J1 pad 4: C5 -> C5_FPGA
- J1 pad 6: +3.3V -> J1_46
- J2 pad 1: +3.3V -> J1_46
- J2 pad 3: A1 -> A1_FPGA
- J2 pad 4: B1 -> B1_FPGA
- J2 pad 5: D1 -> D1_FPGA
- J2 pad 6: E2 -> E2_FPGA
- J3 pad 11: +3.3V -> J1_46
- J3 pad 12: +3.3V -> J1_46
- J4 pad 1: J1_1 -> GND
- J4 pad 10: J1_10 -> /GREEN4
- J4 pad 11: J1_11 -> unconnected-(J4-Pin_11-Pad11)
- J4 pad 12: J1_12 -> /BLUE4
- J4 pad 13: J1_13 -> unconnected-(J4-Pin_13-Pad13)
- J4 pad 14: J1_14 -> unconnected-(J4-Pin_14-Pad14)
- J4 pad 15: J1_15 -> unconnected-(J4-Pin_15-Pad15)
- J4 pad 16: J1_16 -> unconnected-(J4-Pin_16-Pad16)
- J4 pad 17: J1_17 -> Net-(J4-Pin_17)
- J4 pad 18: J1_18 -> unconnected-(J4-Pin_18-Pad18)
- J4 pad 19: J1_19 -> Net-(J4-Pin_19)
- J4 pad 2: J1_1 -> GND
- J4 pad 20: J1_20 -> unconnected-(J4-Pin_20-Pad20)
- J4 pad 21: J1_21 -> /TEMP2
- J4 pad 22: J1_22 -> unconnected-(J4-Pin_22-Pad22)
- J4 pad 23: J1_23 -> /TEMP1
- J4 pad 24: J1_24 -> unconnected-(J4-Pin_24-Pad24)
- J4 pad 25: J1_25 -> /MFB
- J4 pad 26: J1_26 -> unconnected-(J4-Pin_26-Pad26)
- J4 pad 27: J1_27 -> /MCLK1
- J4 pad 28: J1_28 -> unconnected-(J4-Pin_28-Pad28)
- J4 pad 29: J1_29 -> /DT1
- J4 pad 3: J1_3 -> /DATA
- J4 pad 30: J1_30 -> unconnected-(J4-Pin_30-Pad30)
- J4 pad 31: J1_31 -> /SCLK1
- J4 pad 32: J1_32 -> unconnected-(J4-Pin_32-Pad32)
- J4 pad 33: J1_33 -> /RFS1
- J4 pad 34: J1_34 -> unconnected-(J4-Pin_34-Pad34)
- J4 pad 35: J1_35 -> /DR1
- J4 pad 36: J1_36 -> unconnected-(J4-Pin_36-Pad36)
- J4 pad 37: J1_37 -> /CLOCK
- J4 pad 38: J1_38 -> PCM_DOUT_3V3
- J4 pad 39: J1_39 -> /EN_DC
- J4 pad 4: J1_4 -> unconnected-(J4-Pin_4-Pad4)
- J4 pad 40: J1_40 -> /I2C_DATA_1V8
- J4 pad 41: J1_41 -> /MODE
- J4 pad 42: J1_42 -> /I2C_SCL_1V8
- J4 pad 43: J1_43 -> /SEL1V8
- J4 pad 44: J1_44 -> /PETp0
- J4 pad 47: J1_47 -> J1_46
- J4 pad 48: J1_48 -> /I2C1_INT
- J4 pad 49: J1_1 -> GND
- J4 pad 50: J1_1 -> GND
- J4 pad 7: J1_7 -> /LR_SELECT
- J4 pad 8: J1_8 -> /RED4
- J4 pad 9: J1_9 -> unconnected-(J4-Pin_9-Pad9)
- J5 pad 1: J1_1 -> GND
- J5 pad 10: J2_10 -> /BLUE5
- J5 pad 11: J2_11 -> /WCLK
- J5 pad 12: J2_12 -> /CTP_INT
- J5 pad 13: J2_13 -> /I2S_DIN
- J5 pad 14: J2_14 -> /CPT_WAKE
- J5 pad 15: J2_15 -> /I2S_DOUT
- J5 pad 16: J2_16 -> /CPT_SDA
- J5 pad 17: J2_17 -> /V1.8_MODE
- J5 pad 18: J2_18 -> /CPT_SCL
- J5 pad 19: J2_19 -> /SWDIO
- J5 pad 2: J1_1 -> GND
- J5 pad 20: J2_20 -> /GREEN7
- J5 pad 21: J2_21 -> /SWCLK
- J5 pad 22: J2_22 -> /GREEN6
- J5 pad 23: J2_23 -> /PWM
- J5 pad 24: J2_24 -> /GREEN5
- J5 pad 25: J2_25 -> /EXT_SW
- J5 pad 26: J2_26 -> /PIN35
- J5 pad 27: J2_27 -> /SCL
- J5 pad 28: J2_28 -> /DATA_ENABLE
- J5 pad 29: J2_29 -> /SDA
- J5 pad 3: J2_3 -> unconnected-(J5-Pin_3-Pad3)
- J5 pad 30: J2_30 -> /VSYNC
- J5 pad 31: J2_31 -> /SD_DAT1
- J5 pad 32: J2_32 -> /HSYNC
- J5 pad 33: J2_33 -> /SD_PRESENT
- J5 pad 34: J2_34 -> /DISP_ON_OFF
- J5 pad 35: J2_35 -> /SD_DAT0
- J5 pad 36: J2_36 -> /RED7
- J5 pad 37: J2_37 -> /SD_CLK
- J5 pad 38: J2_38 -> /DCLK
- J5 pad 39: J2_39 -> /SD_DAT2
- J5 pad 4: J2_4 -> /BLUE7
- J5 pad 40: J2_40 -> /RED6
- J5 pad 41: J2_41 -> /SD_CMD
- J5 pad 42: J2_42 -> /RED5
- J5 pad 43: J2_43 -> /SD_CD
- J5 pad 44: J2_44 -> /BL_PWM
- J5 pad 47: J2_47 -> /BL_SDA
- J5 pad 48: J2_48 -> /BL_SCL
- J5 pad 49: J1_1 -> GND
- J5 pad 50: J1_1 -> GND
- J5 pad 7: J2_7 -> /I2S_MCLK
- J5 pad 8: J2_8 -> /BLUE6
- J5 pad 9: J2_9 -> /I2S_BCLK
- M1 pad 26: /USIM_VPP -> GND
- M1 pad 31: UART_RX_3V3 -> E2_FPGA
- M1 pad 35: J1_13 -> PCM_DIN_3V3
- M1 pad 4: 3V3 -> Net-(J10-Pin_2)
- M1 pad 40: RI_HOST_WAKE_3V3 -> B3_FPGA
- M1 pad 42: J1_27 -> PCM_CLK_3V3
- M1 pad 43: J1_29 -> PCM_SYNC_3V#
- M1 pad 44: J1_31 -> PCM_CLK_DIR
- M1 pad 52: I2C_DATA_1V8 -> /I2C_DATA_1V8
- M1 pad 53: I2C_SCL_1V8 -> /I2C_SCL_1V8
- M1 pad 54: PETp0 -> /PETp0
- M1 pad 55: PERp0 -> /PERp0
- M10 pad 11: J2_10 -> /SD_DAT2
- M10 pad 15: J2_8 -> /SD_CLK
- M10 pad 18: J2_6 -> /SD_DAT0
- M10 pad 19: J2_4 -> /SD_PRESENT
- M10 pad 20: J2_2 -> /SD_DAT1
- M10 pad 5: /USIM_VPP -> GND
- M10 pad 6: SD_VDD -> /SD_VDD
- M10 pad 8: J2_12 -> /SD_CMD
- M10 pad 9: J2_14 -> /SD_CD
- M11 pad 18: /VALID3 -> //VALID3
- M11 pad 19: /VALID2 -> //VALID2
- M11 pad 20: /VALID1 -> //VALID1
- M11 pad 21: /SHUTDOWN -> //SHUTDOWN
- M11 pad 22: ENABLE -> /ENABLE
- M12 pad 1: VCC_3V3 -> Net-(J8-Pin_2)
- M12 pad 10: TEMP1 -> /TEMP1
- M12 pad 11: TEMP2 -> /TEMP2
- M12 pad 13: UART_TX_IND -> A3_FPGA
- M12 pad 14: UART_CTS -> /UART_CTS
- M12 pad 15: J1_14 -> /SDA
- M12 pad 16: J1_12 -> /SCL
- M12 pad 17: /RESET -> //RESET_BT
- M12 pad 18: GPIO_P2_3 -> /GPIO_P2_3
- M12 pad 19: J2_34 -> /PWM
- M12 pad 20: LED2 -> /LED2
- M12 pad 21: LED1 -> /LED1
- M12 pad 22: UART_RTS -> /UART_RTS
- M12 pad 23: UART_TXD -> B6_FPGA
- M12 pad 24: UART_RXD -> C5_FPGA
- M12 pad 4: DR1 -> /DR1
- M12 pad 5: RFS1 -> /RFS1
- M12 pad 6: SCLK1 -> /SCLK1
- M12 pad 7: DT1 -> /DT1
- M12 pad 8: MCLK1 -> /MCLK1
- M12 pad 9: MFB -> /MFB
- M14 pad 1: VBAT -> Net-(J7-Pin_2)
- M14 pad 12: +3.3V -> Net-(J12-Pin_2)
- M14 pad 13: GPIO1 -> /GPIO1
- M14 pad 15: I2S_DOUT -> /I2S_DOUT
- M14 pad 16: I2S_DIN -> /I2S_DIN
- M14 pad 17: J1_20 -> /WCLK
- M14 pad 18: I2S_BCLK -> /I2S_BCLK
- M14 pad 19: I2S_MCLK -> /I2S_MCLK
- M14 pad 20: J1_14 -> /SDA
- M14 pad 21: J1_12 -> /SCL
- M14 pad 3: /RESET -> //RESET_AUDIO
- M14 pad 4: J1_26 -> /V1.8_MODE
- M15 pad 1: VBAT_OUT -> VBAT
- M3 pad 35: VCC -> /VCC
- M3 pad 41: +3.3V -> J1_46
- M3 pad 45: /UART_TX -> B1_FPGA
- M3 pad 46: /UART_RX -> A1_FPGA
- M4 pad 1: BAT -> Net-(J15-Pin_1)
- M4 pad 10: J2_42 -> /SWDIO
- M4 pad 13: D12 -> /D12
- M4 pad 14: D13 -> /D13
- M4 pad 15: D0 -> /D0
- M4 pad 16: D1 -> /D1
- M4 pad 21: 3V3 -> Net-(J11-Pin_2)
- M4 pad 25: D11 -> /D11
- M4 pad 26: D10 -> /D10
- M4 pad 27: D9 -> /D9
- M4 pad 28: D8 -> /D8
- M4 pad 29: D7 -> /D7
- M4 pad 30: D6 -> /D6
- M4 pad 35: D3 -> /D3
- M4 pad 36: D2 -> /D2
- M4 pad 5: EXT_SW -> /EXT_SW
- M4 pad 7: RST -> /RST_LORA
- M4 pad 9: J2_40 -> /SWCLK
- M5 pad 14: EN -> /EN_DC
- M5 pad 15: J1_8 -> /MODE
- M5 pad 16: J1_6 -> /SEL1V8
- M6 pad 1: LCD_3V3 -> Net-(J9-Pin_2)
- M6 pad 17: DCLK -> /DCLK
- M6 pad 18: DISP_ON_OFF -> /DISP_ON_OFF
- M6 pad 19: HSYNC -> /HSYNC
- M6 pad 20: J2_39 -> /VSYNC
- M6 pad 21: DATA_ENABLE -> /DATA_ENABLE
- M6 pad 23: PIN35 -> /PIN35
- M6 pad 30: CPT_SCL -> /CPT_SCL
- M6 pad 31: CPT_SDA -> /CPT_SDA
- M6 pad 33: CPT_WAKE -> /CPT_WAKE
- M6 pad 34: CTP_INT -> /CTP_INT
- M6 pad 5: BL_SDA -> /BL_SDA
- M6 pad 50: RED4 -> /RED4
- M6 pad 51: J2_32 -> /RED5
- M6 pad 52: J2_30 -> /RED6
- M6 pad 53: J2_28 -> /RED7
- M6 pad 59: GREEN4 -> /GREEN4
- M6 pad 6: BL_SCL -> /BL_SCL
- M6 pad 60: GREEN5 -> /GREEN5
- M6 pad 61: GREEN6 -> /GREEN6
- M6 pad 62: GREEN7 -> /GREEN7
- M6 pad 68: BLUE4 -> /BLUE4
- M6 pad 69: BLUE5 -> /BLUE5
- M6 pad 70: BLUE6 -> /BLUE6
- M6 pad 71: BLUE7 -> /BLUE7
- M6 pad 8: BL_PWM -> /BL_PWM
- M7 pad 1: VCC -> Net-(J6-Pin_2)
- M7 pad 10: DATA -> /DATA
- M7 pad 4: J1_32 -> /LR_SELECT
- M7 pad 6: CLOCK -> /CLOCK
- R1 pad 1: +3V3 -> J1_46
Routing:
- net J1_46: track 0.00 -> 1164.4 mm, vias 1 -> 10
- net /SCL: track 0.00 -> 468.9 mm, vias 0 -> 2
- net /SDA: track 0.00 -> 462.6 mm, vias 0 -> 2
- net VBAT: track 0.00 -> 390.4 mm, vias 0 -> 5
- net +1.8V: track 0.00 -> 389.2 mm, vias 0 -> 5
- net /TEMP2: track 0.00 -> 357.6 mm, vias 0 -> 2
- net /TEMP1: track 0.00 -> 357.1 mm, vias 0 -> 2
- net /PWM: track 0.00 -> 356.8 mm, vias 0 -> 1
- net /MFB: track 0.00 -> 355.4 mm, vias 0 -> 2
- net /MCLK1: track 0.00 -> 354.2 mm, vias 0 -> 2
- net /DT1: track 0.00 -> 351.4 mm, vias 0 -> 2
- net /SCLK1: track 0.00 -> 348.2 mm, vias 0 -> 2
- net /RFS1: track 0.00 -> 347.2 mm, vias 0 -> 2
- net /DR1: track 0.00 -> 345.0 mm, vias 0 -> 2
- net A3_FPGA: track 0.00 -> 324.9 mm, vias 0 -> 2
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- added copper zone on B.Cu, net GND
- added copper zone on F.Cu, net GND
- added copper zone on In1.Cu, net GND
- added copper zone on In2.Cu, net GND
Other:
- board size 311.8 x 203.2 mm -> 299.7 x 198.2 mm
- board text added: "AUDIO CODEC"
- board text added: "AUDIO JACK"
- board text added: "BAT"
- board text added: "BLUETOOTH"
- board text added: "CELULAR"
- board text added: "DC/DC"
- board text added: "INPUT POWER SELECTOR"
- board text added: "LCD"
- board text added: "LORA"
- board text added: "MIC"
- board text added: "MPPT SOLAR"
- board text added: "SIM/SD"
- board text added: "SOLAR"
- board text added: "USB"
- board text removed: "0"
- board text removed: "0 mm"
- board text removed: "0.0152 mm"
- board text removed: "0.01524 mm"
- board text removed: "0.02"
- board text removed: "0.035 mm"
- board text removed: "0.2104 mm"
- board text removed: "1"
- board text removed: "1.065 mm"
- board text removed: "3.8"
- board text removed: "4.4"
- board text removed: "4.43"
- board text removed: "B.Cu"
- board text removed: "B.Mask"
- board text removed: "B.Paste"
- board text removed: "B.Silkscreen"
- board text removed: "Bottom Silk Screen"
- board text removed: "Bottom Solder Mask"
- board text removed: "Bottom Solder Paste"
- board text removed: "Color"
- board text removed: "Dielectric 1"
- board text removed: "Dielectric 2"
- board text removed: "Dielectric 3"
- board text removed: "Direct Printing"
- board text removed: "Epsilon R"
- board text removed: "F.Cu"
- board text removed: "F.Mask"
- board text removed: "F.Paste"
- board text removed: "F.Silkscreen"
- board text removed: "FR4 natural"
- board text removed: "Green"
- board text removed: "In1.Cu"
- board text removed: "In2.Cu"
- board text removed: "JLCPCB Soldermask"
- board text removed: "Layer Name"
- board text removed: "Loss Tangent"
- board text removed: "Material"
- board text removed: "Nan Ya Plastics NP-155F 7628"
- board text removed: "Nan Ya Plastics NP-155F Core"
- board text removed: "Thickness (mm)"
- board text removed: "Top Silk Screen"
- board text removed: "Top Solder Mask"
- board text removed: "Top Solder Paste"
- board text removed: "Type"
- board text removed: "White"
- board text removed: "copper"
- board text removed: "core"
- board text removed: "prepreg"

Commit message: Fully routing base board
Parts:
- added J20: DC/DC_VOUT, Connector_PinSocket_2.54mm:PinSocket_1x02_P2.54mm_Vertical, F.Cu at (281.0, 262.9)
- added J22: IPS_VOUT, Connector_PinSocket_2.54mm:PinSocket_1x02_P2.54mm_Vertical, F.Cu at (358.5, 197.8)
- added J23: DC/DC_VOUT, Connector_PinSocket_2.54mm:PinSocket_1x02_P2.54mm_Vertical, F.Cu at (411.9, 163.7)
- added J24: IPS_VOUT, Connector_PinSocket_2.54mm:PinSocket_1x02_P2.54mm_Vertical, F.Cu at (416.0, 229.1)
- added J25: DC/DC_VOUT, Connector_PinSocket_2.54mm:PinSocket_1x02_P2.54mm_Vertical, F.Cu at (211.8, 196.2)
- added M16: ~, MegaCastle:MegaCastle2x11-I15.7x23.1-MA0780C-EDGE, F.Cu at (197.8, 161.2)
- added M2: ~, MegaCastle:MegaCastle2x8-I15.0x15.5-M8187, F.Cu at (165.9, 161.6)
- moved J6 20.7 mm to (199.7, 296.1)
Connections:
- net /MODE renamed MODE
- net RESERVED_PIN19 renamed /RESERVED_PIN19
- M11 pad 25: VOUT -> Net-(J22-Pin_2)
- M3 pad 23: /Input -> VOUT
- M3 pad 41: J1_46 -> Net-(J24-Pin_1)
- M5 pad 9: VOUT -> /SEL1V8
Routing:
- net Net-(J23-Pin_1): track 0.00 -> 322.4 mm, vias 0 -> 1
- net VBAT: track 390.4 -> 602.2 mm, vias 5 -> 6
- net /EN_DC: track 138.4 -> 321.5 mm, vias 0 -> 4
- net MODE: track 134.2 -> 291.2 mm, vias 0 -> 4
- net Net-(J25-Pin_1): track 0.00 -> 65.1 mm, vias 0 -> 1
- net /SEL1V8: track 129.4 -> 170.4 mm, vias 0 -> 2
- net J1_46: track 1164.4 -> 1126.4 mm, vias 10 -> 11
- net +1.8V: track 389.2 -> 424.8 mm
- net VOUT: track 187.2 -> 162.4 mm
- net PCM_DIN_3V3: track 313.5 -> 331.1 mm
- net Net-(J6-Pin_2): track 12.9 -> 29.7 mm
- net Net-(J24-Pin_1): track 0.00 -> 14.5 mm
- net Net-(J22-Pin_2): track 0.00 -> 6.48 mm
- net GND: track 76.9 -> 81.0 mm, vias 40 -> 267
- net A3_FPGA: track 324.9 -> 326.8 mm
Other:
- board text added: "${project_name} ${project_version}"
- board text added: "1V8"
- board text added: "1V8/3V3 AudioCDC"
- board text added: "AudioCDC_VBAT"
- board text added: "BT_3V3"
- board text added: "Celular 3V3"
- board text added: "DC/DC 3V3"
- board text added: "DC/DC HE"
- board text added: "DC/DC VOUT"
- board text added: "DC/DC_VOUT"
- board text added: "FPGA_VCCIO"
- board text added: "I2C1_VCC"
- board text added: "I2C2_VCC"
- board text added: "I2C3_VCC"
- board text added: "IPS_VOUT"
- board text added: "LCD module"
- board text added: "LCD_VCC"
- board text added: "LORA_3V3"
- board text added: "LORA_BAT"
- board text added: "MIC_VCC"
- board text added: "SD_VCC"
- board text added: "UART_TX_3V3"
