File: modules/main-carrier/main-carrier.kicad_pcb (KiCad board)
At the start: 4 copper layers, 299.7 x 198.2 mm, 70 parts, among them IC1 PCA9535DW, IC2 PCA9535DW, IC3 PCA9535DW, J1 Conn_01x06_Pin, J10 CELULAR_3V3, J11 LORA_3V3, J12 AudioCDC_VCC, J13 SD_VCC, J14 SIM_VCC, J15 LORA_BAT, J16 I2C1_VCC, J17 FPGA_VCCIO, J18 I2C1_VCC, J19 I2C1_VCC, J2 Conn_01x06_Pin, J20 DC/DC_VOUT, J21 UART_CELL, J22 IPS_VOUT, J23 DC/DC_VOUT, J24 IPS_VOUT, J25 DC/DC_VOUT, J3 Conn_02x06_Odd_Even, J4 Conn_02x25_Odd_Even, J5 Conn_02x25_Odd_Even, J6 Mic_VCC, J7 AudioCDC_VBAT, J8 BT_3V3, J9 LCD_3V3, Q1 BSS138, Q2 BSS138

Commit message: All updates in v1.1
Parts:
- J16: value I2C1_VCC -> I2C2_VCC
- J18: value I2C1_VCC -> I2C3_VCC
- moved FID3 8.52 mm to (129.6, 295.9)
- moved M9 2.74 mm to (371.7, 278.2), turned to 180 degrees
- moved M15 0.83 mm to (339.1, 287.5), turned to 180 degrees
- moved M16 0.75 mm to (198.5, 161.4)
- turned M10 to 180 degrees
- turned M13 to 180 degrees
Routing:
- net VOUT: track 162.4 -> 60.0 mm
- net DIRTY_DC_+: track 82.3 -> 165.2 mm
- net /EN_DC: track 321.5 -> 377.7 mm
- net INTERNAL_SOLAR_IN: track 107.1 -> 55.6 mm
- net Net-(J22-Pin_2): track 6.48 -> 55.1 mm
- net //VALID2: track 29.0 -> 76.9 mm, vias 0 -> 2
- net //VALID1: track 28.5 -> 76.3 mm, vias 0 -> 2
- net /ENABLE: track 27.4 -> 75.1 mm, vias 0 -> 2
- net //SHUTDOWN: track 27.9 -> 75.2 mm, vias 0 -> 2
- net //VALID3: track 29.5 -> 76.5 mm, vias 0 -> 2
- net DIRTY_DC_-: track 96.8 -> 142.9 mm
- net /SD_CD: track 71.8 -> 106.6 mm, vias 0 -> 2
- net /USIM_DATA: track 67.0 -> 99.2 mm, vias 0 -> 1
- net /SDA: track 462.6 -> 494.7 mm
- net /SCL: track 468.9 -> 498.2 mm
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Other:
- board text added: "MIRRORED/FIXED"
- board text added: "ROTATED/FIXED"
