File: modules/main-carrier/main-carrier.kicad_sch (KiCad schematic)
At the start: 29 parts

Commit message: connecting power
Connections:
- net +20V is gone; now on net USB-C_POWER_IN: M8.26
- net VBAT_+ is gone; now on net VBAT_OUT: M15.1
- net VBAT_- is gone; now on net GND: M15.5 (GND)
- net VBAT_OUT: no longer M3.1 (VCC)
Other:
- note added: "AUDIO CODEC"
- note added: "BAT CONNECTOR"
- note added: "CELULAR"
- note added: "INPUT POWER SELECTOR"
- note added: "LCD"
- note added: "SIM/SD"
- moved on the sheet: M11, M15, M3, M5, M7, M8, M9

Commit message: Baseboard SCH update
Connections:
- net INTERNAL_SOLAR_+ is gone; now on net INTERNAL_SOLAR_IN: M9.24
- net J1_1 is gone; now on net EN: M2.3
- net J1_10 is gone; now on net EN: M2.48
- net J1_19 is gone; now on net COEX_UART_TX_3V3: M2.12
- net J1_20 is gone; now on net ENABLE: M2.43
- net J1_26 is gone; now on net I2S_MCLK: M2.40
- net J1_28 is gone; now on net I2S_BCLK: M2.39
- net J1_3 is gone; now on net COEX_UART_RX_3V3: M2.4
- net J1_32 is gone; now on net I2S_DIN: M2.37
- net J1_34 is gone; now on net I2S_DOUT: M2.36
- net J1_36 is gone; now on net GPIO1: M2.35
- net J1_42 is gone; now on net DATA: M2.32
- net J1_44 is gone; now on net CLOCK: M2.31
- net J1_45 is gone; now on net I2C_DATA_1V8: M2.25
- net J1_47 is gone; now on net I2C_SCL_1V8: M2.26
- net J2_1 is gone; now on net BL_SDA: M2.55
- net J2_11 is gone; now on net DISP_ON_OFF: M2.60
- net J2_13 is gone; now on net HSYNC: M2.61
- net J2_16 is gone; now on net BLUE7: M2.97
- net J2_17 is gone; now on net DATA_ENABLE: M2.63
- net J2_18 is gone; now on net BLUE6: M2.96
- net J2_20 is gone; now on net BLUE5: M2.95
- net J2_22 is gone; now on net BLUE4: M2.94
- net J2_24 is gone; now on net BLUE3: M2.93
- net J2_26 is gone; now on net BLUE2: M2.92
- net J2_28 is gone; now on net BLUE1: M2.91
- net J2_29 is gone; now on net CPT_SCL: M2.69
- net J2_3 is gone; now on net BL_SCL: M2.56
- net J2_30 is gone; now on net BLUE0: M2.90
- net J2_31 is gone; now on net CPT_SDA: M2.70
- net J2_32 is gone; now on net GREEN7: M2.89
- net J2_33 is gone; now on net CPT_VDD: M2.71
- net J2_34 is gone; now on net GREEN6: M2.88
- net J2_35 is gone; now on net CPT_WAKE: M2.72
- net J2_36 is gone; now on net GREEN5: M2.87
- net J2_37 is gone; now on net CTP_INT: M2.73
- net J2_38 is gone; now on net GREEN4: M2.86
- net J2_40 is gone; now on net GREEN3: M2.85
- net J2_42 is gone; now on net GREEN2: M2.84
- net J2_44 is gone; now on net GREEN1: M2.83
- net J2_46 is gone; now on net GREEN0: M2.82
- net J2_5 is gone; now on net BL_3V3: M2.57
- net J2_7 is gone; now on net BL_PWM: M2.58
- net J2_9 is gone; now on net DCLK: M2.59
- net LEFT is gone; now on net 3.5MM_LEFT: M13.6
- net LR_SELECT is gone; now on net J1_46: M7.4
- net MIC is gone; now on net 3.5MM_MIC: M13.9
- net MODE is gone; now on net J1_8: M5.15
- net PCM_CLK_3V3 is gone; now on net J1_27: M1.42
- net PCM_CLK_DIR is gone; now on net J1_31: M1.44
- net PCM_DIN_3V3 is gone; now on net J1_13: M1.35
- net PCM_DOUT_3V3 is gone; now on net J1_25: M1.41
- net PCM_SYNC_3V# is gone; now on net J1_29: M1.43
- net PERp0 is gone; now on net J1_50: M1.55
- net PETp0 is gone; now on net J1_49: M1.54
- net PIN35 is gone; now on net J2_19: M6.23
- net RED0 is gone; now on net J2_39: M6.46
- net RED1 is gone; now on net J2_41: M6.47
- net RED2 is gone; now on net J2_43: M6.48
- net RED3 is gone; now on net J2_45: M6.49
- net RED4 is gone; now on net J2_47: M6.50
- net RED5 is gone; now on net J2_49: M6.51
- net RED6 is gone; now on net J2_50: M6.52
- net RED7 is gone; now on net J2_48: M6.53
- net RESERVED_PIN19 is gone; now on net J1_48: M1.56
- net RESERVED_PIN46 is gone; now on net J1_39: M1.49
- net RESIST_XL is gone; now on net J2_25: M6.27
- net RESIST_XR is gone; now on net J2_21: M6.25
- net RESIST_YD is gone; now on net J2_23: M6.26
- net RESIST_YU is gone; now on net J2_27: M6.28
- net RIGHT is gone; now on net 3.5MM_RIGHT: M13.10
- net RI_HOST_WAKE_3V3 is gone; now on net J1_23: M1.40
- net SCL is gone; now on net J1_22: M12.16, M14.21, M4.32
- net SDA is gone; now on net J1_24: M12.15, M14.20, M4.33
- net SD_CD is gone; now on net J2_14: M10.9
- net SD_CLK is gone; now on net J2_8: M10.15
- net SD_CMD is gone; now on net J2_12: M10.8
- net SD_DAT0 is gone; now on net J2_6: M10.18
- net SD_DAT1 is gone; now on net J2_2: M10.20
- net SD_DAT2 is gone; now on net J2_10: M10.11
- net SD_GND is gone; now on net GND: M10.17
- net SD_PRESENT is gone; now on net J2_4: M10.19
- net SEL1V8 is gone; now on net J1_6: M5.16
- net SIM_CLK is gone; now on net USIM_CLK: M10.13
- net SIM_DATA is gone; now on net USIM_DATA: M10.14
- net SIM_GND is gone; now on net GND: M10.7
- net SIM_RESET is gone; now on net /USIM_RESET: M10.4
- net SIM_VCC is gone; now on net USIM_VDD: M10.3
- net SIM_VPP is gone; now on net USIM_VPP: M10.5
- net UART_CTS_3V3 is gone; now on net J1_7: M1.32
- net UART_RX_3V3 is gone; now on net J1_5: M1.31
- net UART_TX_3V3 is gone; now on net J1_17: M1.37
- net USB_D+ is gone; now on net J1_37: M1.48
- net USB_D- is gone; now on net J1_35: M1.47
- net USIM_SIM_PRESENT_IN is gone; now on net J1_41: M1.50
- net V1.8_MODE is gone; now on net J1_40: M14.4
- net VSYNC is gone; now on net J2_15: M6.20
- net WCLK is gone; now on net J1_30: M14.17
- net /CLKREQ is gone; now on net J1_33: M1.27
- net /DTR_SLEEP_MODE_3V3 is gone; now on net J1_11: M1.34
- net /LED_WWAN_OC_OUT is gone; now on net J1_43: M1.51
- net /RESET is gone; now on net J1_38: M12.17, M14.3
- net /RESET_3V3 is gone; now on net J1_15: M1.36
- net /SHUTDOWN is gone; now on net J1_18: M11.21
- net /VALID1 is gone; now on net J1_16: M11.20
- net /VALID2 is gone; now on net J1_14: M11.19
- net /VALID3 is gone; now on net J1_12: M11.18
- net /WAKE_3V3 is gone; now on net J1_21: M1.39
- net /W_DISABLE_3V3 is gone; now on net J1_9: M1.33
- net USIM_DATA: now also M1.23
- net /USIM_RESET: now also M1.25
- no-connect marks 13 -> 16
Other:
- note added: "AUDIO"
- note added: "All to FPGA"
- note added: "FPGA LEFT"
- note added: "FPGA RIGHT"
- note added: "LCD_LEFT"
- note added: "LCD_RIGHT"
- note added: "MPPT SOLAR"
- note added: "MicroSIM connectedto CELULAR SD needs to be connected to FPGA"
- note added: "PWR SELECTOR"
- note added: "SD"
- note added: "SPEAKER to connector Everything else to FPGA"
- moved on the sheet: M1, M10, M11, M12, M13, M14, M15, M3, M4, M5, M6, M7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

Commit message: Adding icesugar module - placing Ice sugar on base board, remove FPGA as module, add FPGA directly
Parts:
- removed M2: ~, MegaCastle:MegaCastle2x52-I42.0x127.3-M1, symbol MegaCastle:MegaCastle2x52-I42.0x127.3-M1
- added J1, J2: Conn_01x06_Pin, Connector_PinHeader_2.54mm:PinHeader_1x06_P2.54mm_Vertical, symbol Connector:Conn_01x06_Pin
- added J3: Conn_02x06_Odd_Even, Connector_PinHeader_2.54mm:PinHeader_2x06_P2.54mm_Vertical, symbol Connector_Generic:Conn_02x06_Odd_Even
- added J4, J5: Conn_02x25_Odd_Even, Connector_PinHeader_2.54mm:PinHeader_2x25_P2.54mm_Vertical, symbol Connector_Generic:Conn_02x25_Odd_Even
Connections:
- net CPT_SDA is gone; now on net VCCIO: M6.31
- net CTP_INT is gone; now on net GND: M6.34
- net I2C_DATA_1V8 is gone; now on net VCCIO: M1.52
- net J1_6 is gone; now on net VCCIO: M5.16
- net J2_2 is gone; now on net GND: M10.20
- net J2_6 is gone; now on net VCCIO: M10.18
- net +3.3V: now also M12.16, M14.21, J1.6 (Pin_6), J2.1 (Pin_1), J3.11 (Pin_11), J3.12 (Pin_12), J4.12 (Pin_12), J4.46 (Pin_46), J4.5 (Pin_5), J5.36 (Pin_36), J5.46 (Pin_46), J5.5 (Pin_5)
- net BLUE5: now also J5.20 (Pin_20)
- net BLUE6: now also J5.18 (Pin_18)
- net BLUE7: now also J5.16 (Pin_16)
- net BL_PWM: now also J5.31 (Pin_31)
- net BL_SCL: now also J5.29 (Pin_29)
- net BL_SDA: now also J5.27 (Pin_27)
- net CLOCK: now also J4.30 (Pin_30)
- net CPT_SCL: now also J5.43 (Pin_43)
- net CPT_WAKE: now also J5.47 (Pin_47)
- net D1: now also J2.5 (Pin_5)
- net DATA: now also J4.28 (Pin_28)
- net DATA_ENABLE: now also J5.41 (Pin_41)
- net DCLK: now also J5.33 (Pin_33)
- net DISP_ON_OFF: now also J5.35 (Pin_35)
- net EN: now also J4.10 (Pin_10)
- net EXT_SW: now also J5.48 (Pin_48)
- net GND: now also J1.5 (Pin_5), J2.2 (Pin_2), J3.10 (Pin_10), J3.9 (Pin_9), J4.1 (Pin_1), J4.2 (Pin_2), J4.49 (Pin_49), J4.50 (Pin_50), J5.1 (Pin_1), J5.2 (Pin_2), J5.49 (Pin_49), J5.50 (Pin_50)
- net GREEN5: now also J5.26 (Pin_26)
- net GREEN6: now also J5.24 (Pin_24)
- net GREEN7: now also J5.22 (Pin_22)
- net HSYNC: now also J5.37 (Pin_37)
- net I2C_SCL_1V8: now also J4.47 (Pin_47)
- net I2S_BCLK: now also J4.18 (Pin_18)
- net I2S_DIN: now also J4.22 (Pin_22)
- net I2S_DOUT: now also J4.24 (Pin_24)
- net I2S_MCLK: now also J4.16 (Pin_16)
- net J1_11: now also J4.11 (Pin_11); no longer M1.34
- net J1_13: now also J4.13 (Pin_13)
- net J1_14: now also M12.15, M14.20, J4.14 (Pin_14), J5.38 (Pin_38), J5.44 (Pin_44); no longer M11.19
- net J1_15: now also J4.15 (Pin_15); no longer M1.36
- net J1_17: now also J4.17 (Pin_17); no longer M1.37
- net J1_21: now also J4.21 (Pin_21); no longer M1.39
- net J1_23: now also J4.23 (Pin_23); no longer M1.40
- net J1_25: now also J4.25 (Pin_25); no longer M1.41
- net J1_27: now also J4.27 (Pin_27)
- net J1_29: now also J4.29 (Pin_29)
- net J1_31: now also J4.31 (Pin_31)
- net J1_33: now also J4.33 (Pin_33); no longer M1.27
- net J1_35: now also J4.35 (Pin_35); no longer M1.47
- net J1_37: now also J4.37 (Pin_37); no longer M1.48
- net J1_38: now also J4.38 (Pin_38); no longer M12.17, M14.3
- net J1_39: now also J4.39 (Pin_39); no longer M1.49
- net J1_4: now also J4.4 (Pin_4)
- net J1_40: now also J4.40 (Pin_40); no longer M14.4
- net J1_41: now also J4.41 (Pin_41); no longer M1.50
- net J1_43: now also J4.43 (Pin_43); no longer M1.51
- net J1_48: now also J4.48 (Pin_48); no longer M1.56
- net J1_7: now also J4.7 (Pin_7); no longer M1.32
- net J1_8: now also J4.8 (Pin_8)
- net J1_9: now also J4.9 (Pin_9); no longer M1.33
- net J2_10: now also J5.10 (Pin_10)
- net J2_12: now also J5.12 (Pin_12)
- net J2_14: now also J5.14 (Pin_14)
- net J2_15: now also J5.15 (Pin_15); no longer M6.20
- net J2_19: now also J5.19 (Pin_19); no longer M6.23
- net J2_21: now also J5.21 (Pin_21); no longer M6.25
- net J2_23: now also J5.23 (Pin_23); no longer M6.26
- net J2_25: now also J5.25 (Pin_25); no longer M6.27
- net J2_39: now also M6.20, J5.39 (Pin_39); no longer M6.46
- net J2_4: now also J5.4 (Pin_4)
- net J2_8: now also J5.8 (Pin_8)
- net VCCIO: now also J4.45 (Pin_45), J4.6 (Pin_6), J5.45 (Pin_45), J5.6 (Pin_6)
- net J1_12 renamed /VALID3
- net J1_16 renamed /VALID1
- net J1_18 renamed /SHUTDOWN
- removed net J1_22: M12.16, M14.21, M4.32
- removed net J1_24: M12.15, M14.20, M4.33
- net J1_30 renamed J1_20
- net J1_20: now also J4.20 (Pin_20)
- net J1_46 renamed J1_32
- net J1_32: now also J4.32 (Pin_32)
- net J1_49 renamed PETp0
- net J1_5 renamed UART_RX_3V3
- net J1_50 renamed PERp0
- net J2_27 renamed RESIST_YU
- net J2_41 renamed RED1
- net J2_43 renamed RED2
- net J2_45 renamed RED3
- net J2_47 renamed RED4
- net J2_48 renamed J2_28
- net J2_28: now also J5.28 (Pin_28)
- net J2_49 renamed J2_32
- net J2_32: now also J5.32 (Pin_32)
- net J2_50 renamed J2_30
- net J2_30: now also J5.30 (Pin_30)
- net PWM renamed J2_34
- net J2_34: now also J5.34 (Pin_34)
- net SWCLK renamed J2_40
- net J2_40: now also J5.40 (Pin_40)
- net SWDIO renamed J2_42
- net J2_42: now also J5.42 (Pin_42)
- new net A1: J2.3 (Pin_3)
- new net A1_DUP: J3.8 (Pin_8)
- new net A3: J1.2 (Pin_2)
- new net B1: J2.4 (Pin_4)
- new net B1_DUP: J3.7 (Pin_7)
- new net B3: J1.1 (Pin_1)
- new net B4: J3.1 (Pin_1)
- new net B5: J3.3 (Pin_3)
- new net B6: J1.3 (Pin_3)
- new net C2: J3.6 (Pin_6)
- new net C5: J1.4 (Pin_4)
- new net C6: J3.2 (Pin_2)
- new net E1: J3.5 (Pin_5)
- new net E2: J2.6 (Pin_6)
- new net E3: J3.4 (Pin_4)
- new net J1_19: J4.19 (Pin_19)
- new net J1_26: J4.26 (Pin_26), M14.4
- new net J1_3: J4.3 (Pin_3)
- new net J1_34: J4.34 (Pin_34)
- new net J1_36: J4.36 (Pin_36)
- new net J1_42: J4.42 (Pin_42)
- new net J1_44: J4.44 (Pin_44)
- new net J2_11: J5.11 (Pin_11)
- new net J2_13: J5.13 (Pin_13)
- new net J2_17: J5.17 (Pin_17)
- new net J2_3: J5.3 (Pin_3)
- new net J2_7: J5.7 (Pin_7)
- new net J2_9: J5.9 (Pin_9)
- new net PCM_DOUT_3V3: M1.41
- new net PIN35: M6.23
- new net RED0: M6.46
- new net RESERVED_PIN19: M1.56
- new net RESERVED_PIN46: M1.49
- new net RESIST_XL: M6.27
- new net RESIST_XR: M6.25
- new net RESIST_YD: M6.26
- new net RI_HOST_WAKE_3V3: M1.40
- new net UART_CTS_3V3: M1.32
- new net UART_TX_3V3: M1.37
- new net USB_D+: M1.48
- new net USB_D-: M1.47
- new net USIM_SIM_PRESENT_IN: M1.50
- new net /CLKREQ: M1.27
- new net /DTR_SLEEP_MODE_3V3: M1.34
- new net /LED_WWAN_OC_OUT: M1.51
- new net /RESET: M12.17, M14.3
- new net /RESET_3V3: M1.36
- new net /VALID2: M11.19
- new net /WAKE_3V3: M1.39
- new net /W_DISABLE_3V3: M1.33
- no-connect marks 16 -> 15
Other:
- note added: "AUDIO I2C IO"
- note added: "BT"
- note added: "FPGA VCC"
- note added: "LoRa"
- note added: "PWR SELECTOR I2C IO"
- note added: "Why on earth are A1 and B1 connected to two different PMODs, when there are unused pins on the FPGA?"
- note removed: "FPGA"
- note removed: "PWR SELECTOR"
- moved on the sheet: M12

Commit message: Routing
Parts:
- removed LOGO1: Intergalaktik Logo, intergalaktik:intergalaktik, symbol Mechanical:Fiducial
- removed LOGO2: Radiona Logo, radiona:radiona, symbol Mechanical:Fiducial
- added D2, D3: LED_Small, LED_SMD:LED_0603_1608Metric, symbol Device:LED_Small
- added H5, H6, H7, H8: MH, MountingHole:MountingHole_3mm_Pad, symbol Mechanical:MountingHole_Pad
- added IC1, IC2, IC3: PCA9535DW, PCA9535DW:SOIC127P1030X265-24N, symbol PCA9535DW:PCA9535DW
- added J10: CELULAR_3V3, Connector_PinSocket_2.54mm:PinSocket_1x02_P2.54mm_Vertical, symbol Connector:Conn_01x02_Pin
- added J11: LORA_3V3, Connector_PinSocket_2.54mm:PinSocket_1x02_P2.54mm_Vertical, symbol Connector:Conn_01x02_Pin
- added J12: AudioCDC_VCC, Connector_PinSocket_2.54mm:PinSocket_1x03_P2.54mm_Vertical, symbol Connector:Conn_01x03_Pin
- added J13: SD_VCC, Connector_PinSocket_2.54mm:PinSocket_1x03_P2.54mm_Vertical, symbol Connector:Conn_01x03_Pin
- added J14: SIM_VCC, Connector_PinSocket_2.54mm:PinSocket_1x03_P2.54mm_Vertical, symbol Connector:Conn_01x03_Pin
- added J15: LORA_BAT, Connector_PinSocket_2.54mm:PinSocket_1x02_P2.54mm_Vertical, symbol Connector:Conn_01x02_Pin
- added J16, J18, J19: I2C1_VCC, Connector_PinSocket_2.54mm:PinSocket_1x03_P2.54mm_Vertical, symbol Connector:Conn_01x03_Pin
- added J17: FPGA_VCCIO, Connector_PinSocket_2.54mm:PinSocket_1x03_P2.54mm_Vertical, symbol Connector:Conn_01x03_Pin
- added J21: UART_CELL, Connector_PinSocket_2.54mm:PinSocket_1x02_P2.54mm_Vertical, symbol Connector:Conn_01x02_Pin
- added J6: Mic_VCC, Connector_PinSocket_2.54mm:PinSocket_1x03_P2.54mm_Vertical, symbol Connector:Conn_01x03_Pin
- added J7: AudioCDC_VBAT, Connector_PinSocket_2.54mm:PinSocket_1x02_P2.54mm_Vertical, symbol Connector:Conn_01x02_Pin
- added J8: BT_3V3, Connector_PinSocket_2.54mm:PinSocket_1x02_P2.54mm_Vertical, symbol Connector:Conn_01x02_Pin
- added J9: LCD_3V3, Connector_PinSocket_2.54mm:PinSocket_1x02_P2.54mm_Vertical, symbol Connector:Conn_01x02_Pin
- added Q1, Q2: BSS138, Package_TO_SOT_SMD:SOT-23, symbol Transistor_FET:BSS138
- added R2, R3, R4, R5, R6, R7: 10K, Resistor_SMD:R_0603_1608Metric, symbol Device:R
Connections:
- net J1_21 is gone; now on net TEMP2: J4.21 (Pin_21)
- net J1_23 is gone; now on net TEMP1: J4.23 (Pin_23)
- net J1_25 is gone; now on net MFB: J4.25 (Pin_25)
- net J1_3 is gone; now on net DATA: J4.3 (Pin_3)
- net J1_33 is gone; now on net RFS1: J4.33 (Pin_33)
- net J1_35 is gone; now on net DR1: J4.35 (Pin_35)
- net J1_37 is gone; now on net CLOCK: J4.37 (Pin_37)
- net J1_38 is gone; now on net PCM_DOUT_3V3: J4.38 (Pin_38)
- net J1_42 is gone; now on net I2C_SCL_1V8: J4.42 (Pin_42)
- net J1_44 is gone; now on net PETp0: J4.44 (Pin_44)
- net J2_13 is gone; now on net I2S_DIN: J5.13 (Pin_13)
- net J2_15 is gone; now on net I2S_DOUT: J5.15 (Pin_15)
- net J2_25 is gone; now on net EXT_SW: J5.25 (Pin_25)
- net J2_7 is gone; now on net I2S_MCLK: J5.7 (Pin_7)
- net J2_9 is gone; now on net I2S_BCLK: J5.9 (Pin_9)
- net RI_HOST_WAKE_3V3 is gone; now on net B3_FPGA: M1.40
- net UART_RX is gone; now on net A1_FPGA: M3.46
- net UART_RXD is gone; now on net C5_FPGA: M12.24
- net UART_RX_3V3 is gone; now on net E2_FPGA: M1.31
- net UART_TX is gone; now on net B1_FPGA: M3.45
- net UART_TXD is gone; now on net B6_FPGA: M12.23
- net UART_TX_IND is gone; now on net A3_FPGA: M12.13
- net USIM_VPP is gone; now on net GND: M1.26, M10.5
- net VBAT_OUT is gone; now on net VBAT: M15.1
- net +3.3V: now also J4.47 (Pin_47), R1.1, IC2.21 (A0), J10.1 (Pin_1), J11.1 (Pin_1), J12.1 (Pin_1), J13.1 (Pin_1), J14.1 (Pin_1), J16.1 (Pin_1), J17.1 (Pin_1), J18.1 (Pin_1), J19.1 (Pin_1), J6.1 (Pin_1), J8.1 (Pin_1), J9.1 (Pin_1), Q1.1 (G), Q2.1 (G), R3.1, R4.1; no longer J4.12 (Pin_12), J5.36 (Pin_36), M12.16, M14.12, M14.21
- net +3V3: no longer R1.1
- net BAT: now also J15.2 (Pin_2); no longer M4.1 (VCC)
- net BLUE4: now also J4.12 (Pin_12)
- net BLUE5: now also J5.10 (Pin_10); no longer J5.20 (Pin_20)
- net BLUE6: now also J5.8 (Pin_8); no longer J5.18 (Pin_18)
- net BLUE7: now also J5.4 (Pin_4); no longer J5.16 (Pin_16)
- net BL_PWM: now also J5.44 (Pin_44); no longer J5.31 (Pin_31)
- net BL_SCL: now also J5.48 (Pin_48); no longer J5.29 (Pin_29)
- net BL_SDA: now also J5.47 (Pin_47); no longer J5.27 (Pin_27)
- net CLOCK: no longer J4.30 (Pin_30)
- net CPT_SCL: now also J5.18 (Pin_18); no longer J5.43 (Pin_43)
- net CPT_WAKE: now also J5.14 (Pin_14); no longer J5.47 (Pin_47)
- net D0: now also IC1.6 (P02)
- net D1: now also IC1.5 (P01); no longer J2.5 (Pin_5)
- net D10: now also IC1.17 (P14)
- net D11: now also IC1.18 (P15)
- net D12: now also IC1.19 (P16)
- net D13: now also IC1.20 (P17)
- net D2: now also IC1.9 (P05)
- net D3: now also IC1.8 (P04)
- net D6: now also IC1.13 (P10)
- net D7: now also IC1.14 (P11)
- net D8: now also IC1.15 (P12)
- net D9: now also IC1.16 (P13)
- net DATA: no longer J4.28 (Pin_28)
- net DATA_ENABLE: now also J5.28 (Pin_28); no longer J5.41 (Pin_41)
- net DCLK: now also J5.38 (Pin_38); no longer J5.33 (Pin_33)
- net DISP_ON_OFF: now also J5.34 (Pin_34); no longer J5.35 (Pin_35)
- net DT1: now also J4.29 (Pin_29)
- net EN: now also IC1.7 (P03); no longer J4.10 (Pin_10), M5.14
- net ENABLE: now also IC2.13 (P10)
- net EXT_SW: no longer J5.48 (Pin_48)
- net GND: now also H5.1, H6.1, H7.1, H8.1, IC1.12 (GND), IC1.2 (A1), IC1.21 (A0), IC1.3 (A2), IC2.12 (GND), IC2.2 (A1), IC3.12 (GND), IC3.3 (A2), R6.1, R7.1; no longer M10.20, M6.34
- net GPIO1: now also IC2.5 (P01)
- net GPIO_P2_3: now also IC2.19 (P16)
- net GREEN4: now also J4.10 (Pin_10)
- net GREEN5: now also J5.24 (Pin_24); no longer J5.26 (Pin_26)
- net GREEN6: now also J5.22 (Pin_22); no longer J5.24 (Pin_24)
- net GREEN7: now also J5.20 (Pin_20); no longer J5.22 (Pin_22)
- net HSYNC: now also J5.32 (Pin_32); no longer J5.37 (Pin_37)
- net I2C_SCL_1V8: no longer J4.47 (Pin_47)
- net I2S_BCLK: no longer J4.18 (Pin_18)
- net I2S_DIN: no longer J4.22 (Pin_22)
- net I2S_DOUT: no longer J4.24 (Pin_24)
- net I2S_MCLK: no longer J4.16 (Pin_16)
- net LED1: now also D3.2 (A), IC3.13 (P10)
- net LED2: now also D2.2 (A), IC3.14 (P11)
- net MCLK1: now also J4.27 (Pin_27)
- net PERp0: now also IC2.10 (P06)
- net PIN35: now also J5.26 (Pin_26)
- net RED4: now also J4.8 (Pin_8)
- net SCLK1: now also J4.31 (Pin_31)
- net SD_CS: now also IC3.4 (P00)
- net SD_VDD: now also J13.2 (Pin_2)
- net STAT2: now also IC3.5 (P01)
- net UART_CTS: now also IC2.11 (P07)
- net UART_CTS_3V3: now also IC2.7 (P03)
- net UART_RTS: now also IC2.18 (P15)
- net UART_TX_3V3: now also J21.2 (Pin_2)
- net USIM_VDD: now also J14.2 (Pin_2)
- net VBAT: now also J7.1 (Pin_1); no longer M14.1 (VCC)
- net VCC: no longer M7.1 (VCC)
- net VCCIO: now also J17.2 (Pin_2), R2.1, R5.1; no longer M1.52, M10.18, M5.16, M6.31
- net /DTR_SLEEP_MODE_3V3: now also IC2.9 (P05)
- net /RESET_3V3: now also IC2.4 (P00)
- net /SHUTDOWN: now also IC2.14 (P11)
- net /VALID1: now also IC2.15 (P12)
- net /VALID2: now also IC2.16 (P13)
- net /VALID3: now also IC2.17 (P14)
- net /WAKE_3V3: now also IC1.10 (P06)
- net /W_DISABLE_3V3: now also IC2.8 (P04)
- net ~{Charge EN}: now also IC3.6 (P02)
- net 3V3: no longer names the net of M1.4
- net 3V3: now also J10.2 (Pin_2); no longer M4.21
- net A1 renamed A1_FPGA
- net A3 renamed A3_FPGA
- net B1 renamed B1_FPGA
- net B3 renamed B3_FPGA
- net B4 renamed B4_FPGA
- net B5 renamed B5_FPGA
- net B6 renamed B6_FPGA
- net C2 renamed C2_FPGA
- net C5 renamed C5_FPGA
- net C6 renamed C6_FPGA
- net E1 renamed E1_FPGA
- net E2 renamed E2_FPGA
- net E3 renamed E3_FPGA
- net J1_11: no longer names the net of J4.11 (Pin_11)
- net J1_13: no longer names the net of J4.13 (Pin_13)
- net J1_13: no longer M1.35
- removed net J1_14: J4.14 (Pin_14), J5.38 (Pin_38), J5.44 (Pin_44), M12.15, M14.20
- net J1_15: no longer names the net of J4.15 (Pin_15)
- net J1_17: no longer names the net of J4.17 (Pin_17)
- net J1_17: now also Q1.3 (D), R5.2
- net J1_19: no longer names the net of J4.19 (Pin_19)
- net J1_19: now also Q2.3 (D), R2.2
- net J1_20: no longer names the net of J4.20 (Pin_20)
- net J1_20: no longer M14.17
- net J1_26: no longer names the net of J4.26 (Pin_26)
- net J1_26: no longer M14.4
- net J1_27 renamed PCM_CLK_3V3
- net PCM_CLK_3V3: no longer J4.27 (Pin_27)
- net J1_29 renamed PCM_SYNC_3V#
- net PCM_SYNC_3V#: now also Q2.2 (S), R3.2; no longer J4.29 (Pin_29)
- net J1_31 renamed PCM_CLK_DIR
- net PCM_CLK_DIR: no longer J4.31 (Pin_31)
- net J1_32: no longer names the net of J4.32 (Pin_32)
- net J1_32: no longer M7.4
- net J1_34: no longer names the net of J4.34 (Pin_34)
- net J1_36: no longer names the net of J4.36 (Pin_36)
- net J1_39 renamed EN_DC
- net EN_DC: now also M5.14
- net J1_4: no longer names the net of J4.4 (Pin_4)
- net J1_40 renamed I2C_DATA_1V8
- net I2C_DATA_1V8: now also M1.52
- net J1_41 renamed MODE
- net MODE: now also M5.15
- net J1_43 renamed SEL1V8
- net SEL1V8: now also M5.16
- net J1_48 renamed I2C1_INT
- net I2C1_INT: now also IC2.1 (~{INT})
- net J1_7 renamed LR_SELECT
- net LR_SELECT: now also M7.4
- removed net J1_8: J4.8 (Pin_8), M5.15
- net J1_9: no longer names the net of J4.9 (Pin_9)
- net J2_10 renamed SD_DAT2
- net SD_DAT2: now also J5.39 (Pin_39); no longer J5.10 (Pin_10)
- net J2_11 renamed WCLK
- net WCLK: now also M14.17
- net J2_12 renamed CTP_INT
- net CTP_INT: now also M6.34; no longer M10.8
- net J2_14 renamed SD_CD
- net SD_CD: now also J5.43 (Pin_43); no longer J5.14 (Pin_14)
- net J2_17 renamed V1.8_MODE
- net V1.8_MODE: now also M14.4
- net J2_19 renamed SWDIO
- net SWDIO: now also M4.10
- net J2_21 renamed SWCLK
- net SWCLK: now also M4.9
- net J2_23 renamed PWM
- net PWM: now also M12.19
- net J2_28 renamed RED7
- net RED7: now also J5.36 (Pin_36); no longer J5.28 (Pin_28)
- net J2_3: no longer names the net of J5.3 (Pin_3)
- net J2_30 renamed RED6
- net RED6: now also J5.40 (Pin_40); no longer J5.30 (Pin_30)
- net J2_32 renamed RED5
- net RED5: now also J5.42 (Pin_42); no longer J5.32 (Pin_32)
- removed net J2_34: J5.34 (Pin_34), M12.19
- net J2_39 renamed VSYNC
- net VSYNC: now also J5.30 (Pin_30); no longer J5.39 (Pin_39)
- net J2_4 renamed SD_PRESENT
- net SD_PRESENT: now also J5.33 (Pin_33); no longer J5.4 (Pin_4)
- removed net J2_40: J5.40 (Pin_40), M4.9
- removed net J2_42: J5.42 (Pin_42), M4.10
- net J2_8 renamed SD_CLK
- net SD_CLK: now also J5.37 (Pin_37); no longer J5.8 (Pin_8)
- net LCD_3V3: no longer names the net of M6.1 (VCC)
- net LCD_3V3: now also J9.2 (Pin_2)
- net RST renamed RST_LORA
- net RST_LORA: now also IC1.4 (P00)
- net VCC_3V3: no longer names the net of M12.1 (VCC)
- net VCC_3V3: now also J8.2 (Pin_2)
- net /RESET renamed /RESET_AUDIO
- net /RESET_AUDIO: now also IC2.6 (P02); no longer M12.17
- new net: IC2.24 (VCC), IC2.3 (A2), J16.2 (Pin_2)
- new net: D3.1 (K), R7.2
- new net: J6.2 (Pin_2), M7.1 (VCC)
- new net: J15.1 (Pin_1), M4.1 (VCC)
- new net: J12.2 (Pin_2), M14.12
- new net: D2.1 (K), R6.2
- new net: J7.2 (Pin_2), M14.1 (VCC)
- new net: IC1.24 (VCC), J19.2 (Pin_2)
- new net: IC3.2 (A1), IC3.24 (VCC), J18.2 (Pin_2)
- new net: J11.2 (Pin_2), M4.21
- new net +1.8V: J12.3 (Pin_3), J13.3 (Pin_3), J14.3 (Pin_3), J16.3 (Pin_3), J17.3 (Pin_3), J18.3 (Pin_3), J19.3 (Pin_3), J6.3 (Pin_3)
- new net CPT_SDA: J5.16 (Pin_16), M6.31
- new net D1_FPGA: J2.5 (Pin_5), J21.1 (Pin_1)
- new net I2C0_INT: IC1.1 (~{INT})
- new net I2C0_SCL: IC1.22 (SCL), IC2.22 (SCL), IC3.22 (SCL)
- new net I2C0_SDA: IC1.23 (SDA), IC2.23 (SDA), IC3.23 (SDA)
- new net I2C2_INT: IC3.1 (~{INT})
- new net PCM_DIN_3V3: M1.35, Q1.2 (S), R4.2
- new net SCL: J5.27 (Pin_27), M12.16, M14.21
- new net SDA: J5.29 (Pin_29), M12.15, M14.20
- new net SD_CMD: J5.41 (Pin_41), M10.8
- new net SD_DAT0: J5.35 (Pin_35), M10.18
- new net SD_DAT1: J5.31 (Pin_31), M10.20
- new net /RESET_BT: IC2.20 (P17), M12.17
- no-connect marks 15 -> 14
Other:
- note added: "BLUE0"
- note added: "BLUE1"
- note added: "BLUE2"
- note added: "BLUE3"
- note added: "BLUE4"
- note added: "BT will not work on 1.8V"
- note added: "Can be 1.8V or 3V3"
- note added: "GREEN0"
- note added: "GREEN1"
- note added: "GREEN2"
- note added: "GREEN3"
- note added: "GREEN4"
- note added: "J1_1"
- note added: "J1_10"
- note added: "J1_11"
- note added: "J1_12"
- note added: "J1_13"
- note added: "J1_14"
- note added: "J1_15"
- note added: "J1_16"
- note added: "J1_17"
- note added: "J1_18"
- note added: "J1_19"
- note added: "J1_2"
- note added: "J1_20"
- note added: "J1_21"
- note added: "J1_22"
- note added: "J1_23"
- note added: "J1_24"
- note added: "J1_25"
- note added: "J1_26"
- note added: "J1_27"
- note added: "J1_28"
- note added: "J1_29"
- note added: "J1_3"
- note added: "J1_30"
- note added: "J1_31"
- note added: "J1_32"
- note added: "J1_33"
- note added: "J1_34"
- note added: "J1_35"
- note added: "J1_36"
- note added: "J1_37"
- note added: "J1_38"
- note added: "J1_39"
- note added: "J1_4"
- note added: "J1_40"
- note added: "J1_41"
- note added: "J1_42"
- note added: "J1_43"
- note added: "J1_44"
- note added: "J1_45"
- note added: "J1_46"
- note added: "J1_47"
- note added: "J1_48"
- note added: "J1_49"
- note added: "J1_5"
- note added: "J1_50"
- note added: "J1_6"
- note added: "J1_7"
- note added: "J1_8"
- note added: "J1_9"
- note added: "J2_1"
- note added: "J2_10"
- note added: "J2_11"
- note added: "J2_12"
- note added: "J2_13"
- note added: "J2_14"
- note added: "J2_15"
- note added: "J2_16"
- note added: "J2_17"
- note added: "J2_18"
- note added: "J2_19"
- note added: "J2_2"
- note added: "J2_20"
- note added: "J2_21"
- note added: "J2_22"
- note added: "J2_23"
- note added: "J2_24"
- note added: "J2_25"
- note added: "J2_26"
- note added: "J2_27"
- note added: "J2_28"
- note added: "J2_29"
- note added: "J2_3"
- note added: "J2_30"
- note added: "J2_31"
- note added: "J2_32"
- note added: "J2_33"
- note added: "J2_34"
- note added: "J2_35"
- note added: "J2_36"
- note added: "J2_37"
- note added: "J2_38"
- note added: "J2_39"
- note added: "J2_4"
- note added: "J2_40"
- note added: "J2_41"
- note added: "J2_42"
- note added: "J2_43"
- note added: "J2_44"
- note added: "J2_45"
- note added: "J2_46"
- note added: "J2_47"
- note added: "J2_48"
- note added: "J2_49"
- note added: "J2_5"
- note added: "J2_50"
- note added: "J2_6"
- note added: "J2_7"
- note added: "J2_8"
- note added: "J2_9"
- note added: "LCD holder mounting holes"
- note added: "NC"
- note added: "PWR SEL"
- note added: "RED0"
- note added: "RED1"
- note added: "RED2"
- note added: "RED3"
- note added: "RED4"
- note added: "RESIST_XL"
- note added: "RESIST_XR"
- note added: "RESIST_YD"
- note added: "RESIST_YU"
- note added: "VBAT!!! Class-D: 2.7 V–5.5 V (SPLVDD and SPRVDD ≥ AVDD)"
- note added: "VCC can be 1.8V or 3V3"
- note removed: "AUDIO I2C IO"
- note removed: "FPGA LEFT"
- note removed: "FPGA RIGHT"
- note removed: "FPGA VCC"
- note removed: "LCD_LEFT"
- note removed: "LCD_RIGHT"
- note removed: "PWR SELECTOR I2C IO"
- moved on the sheet: D1, FID1, FID2, FID3, FID4, FID5, FID6, H1, H2, H3, H4, J1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

Commit message: Fully routing base board
Parts:
- added J20, J23, J25: DC/DC_VOUT, Connector_PinSocket_2.54mm:PinSocket_1x02_P2.54mm_Vertical, symbol Connector:Conn_01x02_Pin
- added J22, J24: IPS_VOUT, Connector_PinSocket_2.54mm:PinSocket_1x02_P2.54mm_Vertical, symbol Connector:Conn_01x02_Pin
- added M16: ~, MegaCastle:MegaCastle2x11-I15.7x23.1-MA0780C-EDGE, symbol MegaCastle:MegaCastle2x11-Module-I15.7x23.1-MA0780C
- added M2: ~, MegaCastle:MegaCastle2x8-I15.0x15.5-M8187, symbol MegaCastle:MegaCastle2x8-I15.0x15.5-M8187
- J16: value I2C1_VCC -> I2C2_VCC
- J18: value I2C1_VCC -> I2C3_VCC
Connections:
- net Input is gone; now on net VOUT: M3.23
- net +1.8V: now also J20.2 (Pin_2)
- net +3.3V: now also J23.2 (Pin_2), J25.2 (Pin_2); no longer M3.41
- net EN_DC: now also M16.3, M2.14
- net GND: now also M16.11 (GND), M2.8 (GND)
- net MODE: now also M16.22, M2.15
- net SEL1V8: now also M5.9, J20.1 (Pin_1)
- net VBAT: now also J24.2 (Pin_2), M16.1 (VCC), M2.1 (VCC)
- net VOUT: now also J22.1 (Pin_1); no longer M11.25, M5.9
- new net: J23.1 (Pin_1), M2.9
- new net: J25.1 (Pin_1), M16.10, M16.13, M16.21
- new net: J24.1 (Pin_1), M3.41
- new net: J22.2 (Pin_2), M11.25
- new net /5V_SEL: M16.12
- no-connect marks 14 -> 27
Other:
- moved on the sheet: D1, M11, M13, M15, M3, M5, M8, M9, R1
