File: modules/main-carrier/main-carrier.kicad_sch (KiCad schematic)
At the start: 70 parts, among them IC1 PCA9535DW, IC2 PCA9535DW, IC3 PCA9535DW, J1 Conn_01x06_Pin, J10 CELULAR_3V3, J11 LORA_3V3, J12 AudioCDC_VCC, J13 SD_VCC, J14 SIM_VCC, J15 LORA_BAT, J16 I2C2_VCC, J17 FPGA_VCCIO, J18 I2C3_VCC, J19 I2C1_VCC, J2 Conn_01x06_Pin, J20 DC/DC_VOUT, J21 UART_CELL, J22 IPS_VOUT, J23 DC/DC_VOUT, J24 IPS_VOUT, J25 DC/DC_VOUT, J3 Conn_02x06_Odd_Even, J4 Conn_02x25_Odd_Even, J5 Conn_02x25_Odd_Even, J6 Mic_VCC, J7 AudioCDC_VBAT, J8 BT_3V3, J9 LCD_3V3, Q1 BSS138, Q2 BSS138

Commit message: All updates in v1.1
Other:
- moved on the sheet: J17, J4, Q1, Q2, R2, R3, R4, R5
