File: modules/mppt-charge/mppt-charge.kicad_pcb (KiCad board)
At the start: 4 copper layers, 40 x 61 mm, 53 parts, among them Q1 SI7272DP, Q3 2N7002, U2 AP63203WU, U3 ACS712, U4 ACS712, U5 MCP4018

Commit message: All updates in v1.1
Parts:
- U1: value ~ -> BQ24650
Other:
- board text added: "SD CS"
- board text removed: "PWR GND"
