File: modules/mppt-charge/mppt-charge.kicad_sch (KiCad schematic)
At the start: 53 parts, among them Q1 SI7272DP, Q3 2N7002, U2 AP63203WU, U3 ACS712, U4 ACS712, U5 MCP4018

Commit message: All updates in v1.1
Parts:
- A1: Mouser (none) -> 485-4172; Mouser_URL (none) -> https://hr.mouser.com/ProductDetail/Adafruit/4172?qs=unwgFE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
- C13, C14: Mouser (none) -> 621-PDS1040-13; Mouser_URL (none) -> https://hr.mouser.com/ProductDetail/621-PDS1040-13
- D1, D2: Mouser (none) -> 583-BAT54C; Mouser_URL (none) -> https://hr.mouser.com/ProductDetail/Rectron/BAT54C?qs=7pEAo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
- JP1, JP2, M1: now not fitted
- L1: Mouser (none) -> 70-IHLM2525CZER100M0; Mouser_URL (none) -> https://hr.mouser.com/ProductDetail/Vishay-Dale/IHLM2525CZE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
- L2: Mouser (none) -> 70-IFSC1515AHER4R7M0; Mouser_URL (none) -> https://hr.mouser.com/ProductDetail/Vishay-Dale/IFSC1515AHE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
- Q1: Mouser (none) -> 781-SI7272DP-GE3; Mouser_URL (none) -> https://hr.mouser.com/ProductDetail/Vishay-Semiconductors/S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
- Q3: Mouser (none) -> 637-2N7002; Mouser_URL (none) -> https://hr.mouser.com/ProductDetail/Diotec-Semiconductor/2N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
- R5: Mouser (none) -> 71-CRCW25122R00FKTG; Mouser_URL (none) -> https://hr.mouser.com/ProductDetail/Vishay/CRCW25122R00FKTG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
- R7, R8: value 100 -> 130
- RSR1: Mouser (none) -> 755-PMR18EZPFU10L0; Mouser_URL (none) -> https://hr.mouser.com/ProductDetail/ROHM-Semiconductor/PMR1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
- U1: value ~ -> BQ24650; Mouser (none) -> 595-BQ24650RVAR; Mouser_URL (none) -> https://hr.mouser.com/ProductDetail/Texas-Instruments/BQ246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
- U2: Mouser (none) -> 621-AP63203QWU-7; Mouser_URL (none) -> https://hr.mouser.com/ProductDetail/Diodes-Incorporated/AP6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
- U3, U4: Mouser (none) -> 250-71240LLCBTR010B3; Mouser_URL (none) -> https://hr.mouser.com/ProductDetail/Allegro-MicroSystems/AC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
- U5: Mouser (none) -> 579-MCP4018T103ELTY; Mouser_URL (none) -> https://hr.mouser.com/ProductDetail/579-MCP4018T103ELTY
